Commit message: Add lite_pro variant; update lite from CAD; verify actuator joint params
Add the lite_pro full-body humanoid and align actuator-derived joint
parameters across the full-body variants against the actuator manuals
(Actuator-Manuals/). Convention: effort_limit = the manual's peak torque;
armature/friction_loss are sysid priors (not in the manuals).

lite_pro (new; 74 DoF; root pelvis; model-only):
- Generated from the Onshape "Humanoid Pro" assembly via the offline
  --convert path; colliders reused from lite (pelvis.scad -> waist.scad to
  match the new root part).
- Arms Robstride: shoulder_pitch RS02 (17 Nm); shoulder roll/yaw + elbow
  RS00 (14); wrist RS05 (5.5). Legs+waist DM: hip pitch/roll + knee +
  waist_yaw DM-J6248P (97); hip_yaw + ankle yaw/pitch + waist roll/pitch
  DM-J4340P (40); ankle_roll RS05 (5.5). Neck Sitodrive TA40 100:1 (9);
  fingers placeholder.

lite (regenerated from updated export):
- Waist simplified 3-DoF -> 1-DoF (waist_yaw only); now 72 DoF.
- Legs on Robstride: hip/knee RS06 (36), hip_yaw RS02 (17), ankle
  yaw/pitch RS00 (14), ankle_roll RS05 (5.5).

lite_biped: legs aligned to the same Robstride mapping (was stale 97 Nm).

Register lite_pro in CMakeLists; update the README variants table.
All 1376 tests pass.

Co-Authored-By: Claude Opus 4.8 (1M context) <noreply@anthropic.com>
Claude-Session: https://claude.ai/code/session_01KXLFn7xhCYz59LiUie9B9k

File: robots/lite/urdf/lite.urdf (robot description, URDF)
Before this commit: robot lite, 75 links, 74 joints
Links:
- removed link waist_pitch
- removed link waist_yaw
- link chest: mass 3.98764 -> 4.30714
- link left_ankle_pitch: mass 0.136941 -> 0.184118
- link left_ankle_yaw: mass 1.382 -> 1.43174
- link left_elbow_pitch: mass 0.1 -> 0.11
- link left_foot: mass 1.18451 -> 1.20654
- link left_hip_pitch: mass 0.595117 -> 0.619442
- link left_hip_roll: mass 1.12092 -> 1.30369
- link left_hip_yaw: mass 2.10215 -> 2.08958
- link left_knee_pitch: mass 0.389417 -> 0.435399
- link left_shoulder_roll: mass 0.41 -> 0.42
- link left_shoulder_yaw: mass 0.416 -> 0.43
- link left_wrist_yaw: mass 0.6 -> 0.540556
- link neck_roll: mass 0.0779115 -> 0.144705
- link neck_yaw: mass 0.0779115 -> 0.118449
- link pelvis: mass 1.72488 -> 3.97182
- link right_ankle_pitch: mass 0.136941 -> 0.184118
- link right_ankle_yaw: mass 1.382 -> 1.43169
- link right_elbow_pitch: mass 0.1 -> 0.11
- link right_foot: mass 1.1845 -> 1.20654
- link right_hip_pitch: mass 0.595116 -> 0.619423
- link right_hip_roll: mass 1.12092 -> 1.30368
- link right_hip_yaw: mass 2.10215 -> 2.08959
- link right_knee_pitch: mass 0.389417 -> 0.435358
- link right_shoulder_roll: mass 0.41 -> 0.42
- link right_shoulder_yaw: mass 0.416 -> 0.43
- link right_wrist_yaw: mass 0.6 -> 0.54
Joints:
- removed joint waist_pitch
- removed joint waist_roll
- joint left_ankle_pitch: limit lower=-0.785398 upper=0.785398 effort=27.0 velocity=100 -> lower=-0.523599 upper=0.872665 effort=14.0 velocity=100; origin xyz=-0 -0 -0.37 rpy=-1.5708 -0 0 -> xyz=0.01 -0 -0.34 rpy=-1.5708 0 -0
- joint left_ankle_roll: origin xyz=0 0.04 -0 rpy=-0 1.5708 0 -> xyz=-0 0.04 0 rpy=0 1.5708 0
- joint left_ankle_yaw: limit lower=-0.785398 upper=0.785398 effort=27.0 velocity=100 -> lower=-0.785398 upper=0.785398 effort=14.0 velocity=100; origin xyz=-0.015 0 0 rpy=1.5708 -0 -0 -> xyz=-0.015 0 0 rpy=1.5708 0 -0
- joint left_elbow_pitch: origin xyz=0.01 -0 -0.08 rpy=-1.5708 -0 -0 -> xyz=0.01 -0 -0.08 rpy=-1.5708 0 0
- joint left_finger1_j1: origin xyz=0 0.035 0.03 rpy=0.785398 -0 -0 -> xyz=0 0.035 0.03 rpy=0.785398 0 -0
- joint left_finger1_j3: origin xyz=0 0.025 0 rpy=0 1.5708 0 -> xyz=0 0.025 0 rpy=-0 1.5708 0
- joint left_finger1_j4: origin xyz=0 0.025 0 rpy=-0 0 -0 -> xyz=0 0.025 -0 rpy=-0 0 0
- joint left_finger2_j1: origin xyz=-0 0.07 0.015 rpy=-0 0 0 -> xyz=0 0.07 0.015 rpy=-0 0 -0
- joint left_finger2_j2: origin xyz=-0 0.01 -0 rpy=-0 -1.5708 0 -> xyz=0 0.01 0 rpy=-0 -1.5708 0
- joint left_finger2_j4: origin xyz=0 0.025 0 rpy=-0 -0 0 -> xyz=0 0.025 0 rpy=-0 -0 -0
- joint left_finger3_j1: origin xyz=-0 0.075 -0 rpy=-0 -0 0 -> xyz=0 0.075 0 rpy=-0 0 -0
- joint left_finger3_j3: origin xyz=0 0.035 -0 rpy=-0 1.5708 0 -> xyz=0 0.035 0 rpy=0 1.5708 0
- joint left_finger3_j4: origin xyz=0 0.03 0 rpy=-0 0 0 -> xyz=-0 0.03 0 rpy=0 -0 0
- joint left_finger4_j1: origin xyz=0 0.07 -0.015 rpy=-0 0 0 -> xyz=0 0.07 -0.015 rpy=-0 0 -0
- joint left_finger4_j2: origin xyz=0 0.01 -0 rpy=0 -1.5708 0 -> xyz=0 0.01 0 rpy=-0 -1.5708 0
- joint left_finger4_j3: origin xyz=0 0.035 0 rpy=-0 1.5708 0 -> xyz=0 0.035 0 rpy=0 1.5708 0
- joint left_finger4_j4: origin xyz=0 0.025 -0 rpy=0 -0 0 -> xyz=0 0.025 -0 rpy=-0 -0 -0
- joint left_finger5_j1: origin xyz=-0 0.065 -0.03 rpy=-0 -0 0 -> xyz=0 0.065 -0.03 rpy=-0 0 -0
- joint left_finger5_j2: origin xyz=0 0.01 0 rpy=-0 -1.5708 0 -> xyz=-0 0.01 0 rpy=-0 -1.5708 0
- joint left_finger5_j3: origin xyz=-0 0.025 0 rpy=0 1.5708 0 -> xyz=0 0.025 0 rpy=0 1.5708 0
- joint left_finger5_j4: origin xyz=-0 0.02 -0 rpy=-0 -0 0 -> xyz=0 0.02 0 rpy=0 -0 0
- joint left_hip_pitch: limit lower=-2.35619 upper=0.785398 effort=97.0 velocity=100 -> lower=-2.35619 upper=0.785398 effort=36.0 velocity=100; origin xyz=0.02 0.07 0 rpy=-1.74533 -0 0 -> xyz=0.02 0.07 0 rpy=-1.74533 0 0
- joint left_hip_roll: limit lower=-0.349066 upper=1.5708 effort=97.0 velocity=100 -> lower=-0.349066 upper=1.5708 effort=36.0 velocity=100; origin xyz=0 0 0 rpy=1.91986 1.39626 1.5708 -> xyz=-0 0 -0 rpy=1.91986 1.39626 1.5708
- joint left_hip_yaw: limit lower=-1.5708 upper=1.5708 effort=97.0 velocity=100 -> lower=-1.5708 upper=1.5708 effort=17.0 velocity=100; origin xyz=0 -0.0068404 -0.0187939 rpy=-0 -1.22173 1.5708 -> xyz=0 -0.0068404 -0.0187939 rpy=0 -1.22173 1.5708
- joint left_knee_pitch: limit lower=0 upper=2.0944 effort=97.0 velocity=100 -> lower=0 upper=2.35619 effort=36.0 velocity=100; origin xyz=-0.01 -0 -0.33 rpy=-1.5708 0 0 -> xyz=-0.01 0 -0.33 rpy=-1.5708 0 0
- joint left_shoulder_pitch: origin xyz=0.09 0.17 -0.01 rpy=-2.96706 -1.5708 0 -> xyz=-0.03 0.09 0.26 rpy=-1.39626 0 0
- joint left_shoulder_roll: origin xyz=0 0 -0 rpy=1.5708 0.174533 1.5708 -> xyz=0 0 0 rpy=1.5708 0.174533 1.5708
- joint left_shoulder_yaw: origin xyz=-0 0.12 -0 rpy=1.5708 -1.5708 0 -> xyz=0 0.12 0 rpy=1.5708 -1.5708 0
- joint left_wrist_pitch: origin xyz=-0 0 0 rpy=0 1.5708 0 -> xyz=0 0 0 rpy=0 1.5708 0
- joint left_wrist_roll: origin xyz=0 0 -0.135 rpy=-1.5708 -0 0 -> xyz=0 -0 -0.135 rpy=-1.5708 0 0
- joint left_wrist_yaw: limit lower=-1.5708 upper=1.5708 effort=5.5 velocity=100 -> lower=-2.0944 upper=1.5708 effort=5.5 velocity=100; origin xyz=-0.01 0.055 0 rpy=1.5708 0 -0 -> xyz=-0.01 0.055 0 rpy=1.5708 -0 -0
- joint neck_pitch: limit lower=-0.523599 upper=0.523599 effort=10 velocity=100 -> lower=-0.698132 upper=0.349066 effort=9.0 velocity=100; origin xyz=0 0.03 -0 rpy=-0 1.5708 0 -> xyz=0 0.0464025 -0.0132592 rpy=-0 1.5708 0
- joint neck_roll: limit lower=-0.523599 upper=0.523599 effort=10 velocity=100 -> lower=-0.523599 upper=0.523599 effort=9.0 velocity=100; origin xyz=0 -0 0.03 rpy=1.5708 0 1.5708 -> xyz=-0.0125027 -0 0.0709062 rpy=1.5708 0 1.5708
- joint neck_yaw: limit lower=-0.785398 upper=0.785398 effort=10 velocity=100 -> lower=-0.785398 upper=0.785398 effort=9.0 velocity=100; origin xyz=0 0.23 -0.02 rpy=-1.5708 -1.5708 0 -> xyz=-0.04 0 0.32 rpy=0 0.174533 0
- joint right_ankle_pitch: limit lower=-0.785398 upper=0.785398 effort=27.0 velocity=100 -> lower=-0.523599 upper=0.872665 effort=14.0 velocity=100; origin xyz=0 0 -0.37 rpy=-1.5708 -0 -0 -> xyz=0.01 0 -0.34 rpy=-1.5708 -0 -0
- joint right_ankle_roll: origin xyz=0 0.05 0 rpy=0 1.5708 0 -> xyz=0 0.04 0 rpy=0 1.5708 0
- joint right_ankle_yaw: limit lower=-0.785398 upper=0.785398 effort=27.0 velocity=100 -> lower=-0.785398 upper=0.785398 effort=14.0 velocity=100; origin xyz=-0.015 0 0 rpy=1.5708 0 -0 -> xyz=-0.015 0 0 rpy=1.5708 -0 -0
- joint right_elbow_pitch: origin xyz=0.01 0 -0.08 rpy=-1.5708 0 0 -> xyz=0.01 0 -0.08 rpy=-1.5708 -0 0
- joint right_finger1_j1: origin xyz=0 0.035 0.03 rpy=0.785398 -0 0 -> xyz=0 0.035 0.03 rpy=0.785398 0 -0
- joint right_finger1_j2: origin xyz=-0 0.01 0 rpy=-0 1.5708 0 -> xyz=0 0.01 0 rpy=-0 1.5708 0
- joint right_finger1_j3: origin xyz=0 0.025 0 rpy=0 -1.5708 0 -> xyz=-0 0.025 -0 rpy=-0 -1.5708 0
- joint right_finger1_j4: origin xyz=0 0.025 -0 rpy=-0 0 -0 -> xyz=0 0.025 -0 rpy=-0 -0 0
- joint right_finger2_j1: origin xyz=-0 0.07 0.015 rpy=0 0 0 -> xyz=0 0.07 0.015 rpy=0 0 -0
- joint right_finger2_j2: origin xyz=-0 0.01 0 rpy=-0 1.5708 0 -> xyz=0 0.01 0 rpy=0 1.5708 0
- joint right_finger2_j4: origin xyz=-0 0.025 -0 rpy=-0 0 -0 -> xyz=0 0.025 0 rpy=0 0 -0
- joint right_finger3_j1: origin xyz=0 0.075 0 rpy=0 0 0 -> xyz=0 0.075 -0 rpy=0 0 -0
- joint right_finger3_j2: origin xyz=-0 0.01 0 rpy=-0 1.5708 0 -> xyz=-0 0.01 0 rpy=0 1.5708 0
- joint right_finger3_j3: origin xyz=-0 0.035 0 rpy=-0 -1.5708 0 -> xyz=0 0.035 0 rpy=0 -1.5708 0
- joint right_finger3_j4: origin xyz=0 0.03 -0 rpy=0 0 -0 -> xyz=0 0.03 -0 rpy=-0 0 -0
- joint right_finger4_j1: origin xyz=0 0.07 -0.015 rpy=0 0 0 -> xyz=0 0.07 -0.015 rpy=0 0 -0
- joint right_finger4_j2: origin xyz=-0 0.01 0 rpy=-0 1.5708 0 -> xyz=0 0.01 -0 rpy=-0 1.5708 0
- joint right_finger4_j3: origin xyz=-0 0.035 0 rpy=0 -1.5708 0 -> xyz=0 0.035 0 rpy=0 -1.5708 0
- joint right_finger4_j4: origin xyz=-0 0.025 0 rpy=0 -0 0 -> xyz=0 0.025 0 rpy=-0 -0 -0
- joint right_finger5_j1: origin xyz=0 0.065 -0.03 rpy=-0 0 0 -> xyz=0 0.065 -0.03 rpy=0 0 -0
- joint right_finger5_j2: origin xyz=-0 0.01 0 rpy=-0 1.5708 0 -> xyz=0 0.01 0 rpy=0 1.5708 0
- joint right_finger5_j3: origin xyz=0 0.025 0 rpy=-0 -1.5708 0 -> xyz=0 0.025 -0 rpy=-0 -1.5708 0
- joint right_finger5_j4: origin xyz=0 0.02 0 rpy=0 0 -0 -> xyz=0 0.02 0 rpy=-0 -0 0
- joint right_hip_pitch: limit lower=-2.35619 upper=0.785398 effort=97.0 velocity=100 -> lower=-2.35619 upper=0.785398 effort=36.0 velocity=100
- joint right_hip_roll: limit lower=-1.5708 upper=0.349066 effort=97.0 velocity=100 -> lower=-1.5708 upper=0.349066 effort=36.0 velocity=100; origin xyz=0 0 -0 rpy=-1.22173 1.39626 -1.5708 -> xyz=0 -0 -0 rpy=-1.22173 1.39626 -1.5708
- joint right_hip_yaw: limit lower=-1.5708 upper=1.5708 effort=97.0 velocity=100 -> lower=-1.5708 upper=1.5708 effort=17.0 velocity=100
- joint right_knee_pitch: limit lower=0 upper=2.0944 effort=97.0 velocity=100 -> lower=0 upper=2.35619 effort=36.0 velocity=100; origin xyz=-0.01 0 -0.33 rpy=-1.5708 0 0 -> xyz=-0.01 -0 -0.33 rpy=-1.5708 0 -0
- joint right_shoulder_pitch: origin xyz=-0.09 0.17 -0.01 rpy=2.96706 -1.5708 0 -> xyz=-0.03 -0.09 0.26 rpy=-1.74533 -0 -0
- joint right_shoulder_yaw: origin xyz=0 0.12 -0 rpy=1.5708 -1.5708 0 -> xyz=-0 0.12 0 rpy=1.5708 -1.5708 0
- joint right_wrist_pitch: origin xyz=0 0 0 rpy=0 1.5708 0 -> xyz=0 0 0 rpy=-0 1.5708 0
- joint right_wrist_roll: origin xyz=0 0 -0.135 rpy=-1.5708 0 0 -> xyz=-0 -0 -0.135 rpy=-1.5708 0 0
- joint right_wrist_yaw: limit lower=-1.5708 upper=1.5708 effort=5.5 velocity=100 -> lower=-1.5708 upper=2.0944 effort=5.5 velocity=100; origin xyz=-0.01 0.055 -0 rpy=1.5708 0 -0 -> xyz=-0.01 0.055 0 rpy=1.5708 -0 -0
- joint waist_yaw: child waist_yaw -> chest; limit lower=-1.5708 upper=1.5708 effort=10 velocity=100 -> lower=-1.5708 upper=1.5708 effort=36.0 velocity=100; origin xyz=0.01 -0 0.1 rpy=-0 0 0 -> xyz=0.02 -0 0.1 rpy=0 -0 0
