Commit message: Add lite_pro variant; update lite from CAD; verify actuator joint params
Add the lite_pro full-body humanoid and align actuator-derived joint
parameters across the full-body variants against the actuator manuals
(Actuator-Manuals/). Convention: effort_limit = the manual's peak torque;
armature/friction_loss are sysid priors (not in the manuals).

lite_pro (new; 74 DoF; root pelvis; model-only):
- Generated from the Onshape "Humanoid Pro" assembly via the offline
  --convert path; colliders reused from lite (pelvis.scad -> waist.scad to
  match the new root part).
- Arms Robstride: shoulder_pitch RS02 (17 Nm); shoulder roll/yaw + elbow
  RS00 (14); wrist RS05 (5.5). Legs+waist DM: hip pitch/roll + knee +
  waist_yaw DM-J6248P (97); hip_yaw + ankle yaw/pitch + waist roll/pitch
  DM-J4340P (40); ankle_roll RS05 (5.5). Neck Sitodrive TA40 100:1 (9);
  fingers placeholder.

lite (regenerated from updated export):
- Waist simplified 3-DoF -> 1-DoF (waist_yaw only); now 72 DoF.
- Legs on Robstride: hip/knee RS06 (36), hip_yaw RS02 (17), ankle
  yaw/pitch RS00 (14), ankle_roll RS05 (5.5).

lite_biped: legs aligned to the same Robstride mapping (was stale 97 Nm).

Register lite_pro in CMakeLists; update the README variants table.
All 1376 tests pass.

Co-Authored-By: Claude Opus 4.8 (1M context) <noreply@anthropic.com>
Claude-Session: https://claude.ai/code/session_01KXLFn7xhCYz59LiUie9B9k

File: robots/lite/xacro/lite.description.xacro (robot description, xacro)
@@ -12,11 +12,11 @@
     <link name="pelvis">
       <inertial>
-        <origin xyz="0.0185085 1.026e-09 0.0225234" rpy="0 0 0" />
-        <mass value="1.72488" />
-        <inertia ixx="0.00450013" ixy="-7.22e-10" ixz="0.000138837" iyy="0.00310923" iyz="5.14e-10" izz="0.00364534" />
+        <origin xyz="0.0135183 5.78646e-07 0.0691358" rpy="0 0 0" />
+        <mass value="3.97182" />
+        <inertia ixx="0.0186861" ixy="7.2433e-08" ixz="-0.000228382" iyy="0.015546" iyz="-9.5463e-08" izz="0.0121371" />
       </inertial>
       <!-- Part pelvis_parts -->
       <collision>
-        <origin xyz="0.02 0 0" rpy="1.5708 1.5708 0" />
+        <origin xyz="0.02 0 -0" rpy="1.5708 1.5708 0" />
         <geometry>
           <cylinder length="0.16" radius="0.05" />
@@ -24,10 +24,10 @@
       </collision>
       <visual>
-        <origin xyz="0.0185085 1.026e-09 0.0225234" rpy="0 -0 0" />
+        <origin xyz="0.0135183 5.78646e-07 0.0691358" rpy="0 -0 0" />
         <geometry>
           <mesh filename="${mesh_root}/pelvis_visual.stl" />
         </geometry>
         <material name="pelvis_parts_material">
-          <color rgba="0.615686 0.811765 0.929412 1" />
+          <color rgba="0.933333 0.933333 0.933333 1" />
         </material>
       </visual>
@@ -36,16 +36,16 @@
     <link name="left_hip_pitch">
       <inertial>
-        <origin xyz="-0.0102357 0.00373281 0.0191791" rpy="0 0 0" />
-        <mass value="0.595117" />
-        <inertia ixx="0.000596324" ixy="5.6211e-05" ixz="-0.000110867" iyy="0.000729574" iyz="4.15124e-05" izz="0.000918625" />
+        <origin xyz="-0.0114774 0.00418673 0.0187959" rpy="0 0 0" />
+        <mass value="0.619442" />
+        <inertia ixx="0.000652303" ixy="5.37205e-05" ixz="-0.00011886" iyy="0.000778993" iyz="4.47861e-05" izz="0.000986073" />
       </inertial>
       <!-- Part left_hip_pitch_parts -->
       <visual>
-        <origin xyz="-0.0102357 0.00373281 0.0191791" rpy="1.74533 0 0" />
+        <origin xyz="-0.0114774 0.00418673 0.0187959" rpy="1.74533 0 -0" />
         <geometry>
           <mesh filename="${mesh_root}/left_hip_pitch_visual.stl" />
         </geometry>
         <material name="left_hip_pitch_parts_material">
-          <color rgba="0.498039 0.498039 0.498039 1" />
+          <color rgba="0.933333 0.933333 0.933333 1" />
         </material>
       </visual>
@@ -54,11 +54,11 @@
     <link name="left_hip_roll">
       <inertial>
-        <origin xyz="-6.4164e-08 0.055907 -0.065773" rpy="0 0 0" />
-        <mass value="1.12092" />
-        <inertia ixx="0.0029112" ixy="5.717e-09" ixz="-8.323e-09" iyy="0.00148103" iyz="-0.000661072" izz="0.00295542" />
+        <origin xyz="-4.8952e-08 0.0525082 -0.0652484" rpy="0 0 0" />
+        <mass value="1.30369" />
+        <inertia ixx="0.00368883" ixy="-7.197e-09" ixz="4.838e-09" iyy="0.00199601" iyz="-0.000913168" izz="0.00358153" />
       </inertial>
       <!-- Part left_hip_roll_parts -->
       <collision>
-        <origin xyz="0 0.181098 -0.0871979" rpy="1.22173 -0 -0" />
+        <origin xyz="0 0.181098 -0.0871979" rpy="1.22173 -0 0" />
         <geometry>
           <cylinder length="0.15" radius="0.05" />
@@ -66,10 +66,10 @@
       </collision>
       <visual>
-        <origin xyz="-6.4164e-08 0.055907 -0.065773" rpy="-0 -1.22173 1.5708" />
+        <origin xyz="-4.8952e-08 0.0525082 -0.0652484" rpy="0 -1.22173 1.5708" />
         <geometry>
           <mesh filename="${mesh_root}/left_hip_roll_visual.stl" />
         </geometry>
         <material name="left_hip_roll_parts_material">
-          <color rgba="0.647059 0.647059 0.647059 1" />
+          <color rgba="0.933333 0.933333 0.933333 1" />
         </material>
       </visual>
@@ -78,16 +78,16 @@
     <link name="left_hip_yaw">
       <inertial>
-        <origin xyz="-0.00141351 -3.74707e-05 -0.232605" rpy="0 0 0" />
-        <mass value="2.10215" />
-        <inertia ixx="0.0106161" ixy="2.40268e-06" ixz="-0.000364568" iyy="0.0108723" iyz="8.54712e-07" izz="0.00262072" />
+        <origin xyz="0.00130442 -2.2783e-05 -0.237299" rpy="0 0 0" />
+        <mass value="2.08958" />
+        <inertia ixx="0.0116205" ixy="1.09303e-06" ixz="-0.000458028" iyy="0.0118686" iyz="2.21073e-07" izz="0.00261694" />
       </inertial>
       <!-- Part left_hip_yaw_parts -->
       <visual>
-        <origin xyz="-0.00141351 -3.74707e-05 -0.232605" rpy="-0 -0 -0" />
+        <origin xyz="0.00130442 -2.2783e-05 -0.237299" rpy="-0 0 -0" />
         <geometry>
           <mesh filename="${mesh_root}/left_hip_yaw_visual.stl" />
         </geometry>
         <material name="left_hip_yaw_parts_material">
-          <color rgba="0.917647 0.917647 0.917647 1" />
+          <color rgba="0.933333 0.933333 0.933333 1" />
         </material>
       </visual>
@@ -96,11 +96,11 @@
     <link name="left_knee_pitch">
       <inertial>
-        <origin xyz="-0.00531998 0.0299356 3.86127e-06" rpy="0 0 0" />
-        <mass value="0.389417" />
-        <inertia ixx="0.000727371" ixy="4.24751e-05" ixz="-2.14082e-06" iyy="0.000543207" iyz="-3.24942e-07" izz="0.000490238" />
+        <origin xyz="-0.00486713 0.0372163 -0.000224083" rpy="0 0 0" />
+        <mass value="0.435399" />
+        <inertia ixx="0.000913317" ixy="6.65453e-05" ixz="-2.2735e-07" iyy="0.000625586" iyz="1.07178e-06" izz="0.000714736" />
       </inertial>
       <!-- Part left_knee_pitch_parts -->
       <collision>
-        <origin xyz="-0.01 0.17 -0" rpy="1.5708 1.5708 0" />
+        <origin xyz="-0.01 0.17 0" rpy="1.5708 1.5708 0" />
         <geometry>
           <cylinder length="0.16" radius="0.045" />
@@ -108,10 +108,10 @@
       </collision>
       <visual>
-        <origin xyz="-0.00531998 0.0299356 3.86127e-06" rpy="1.5708 0 -0" />
+        <origin xyz="-0.00486713 0.0372163 -0.000224083" rpy="1.5708 0 0" />
         <geometry>
           <mesh filename="${mesh_root}/left_knee_pitch_visual.stl" />
         </geometry>
         <material name="left_knee_pitch_parts_material">
-          <color rgba="0.768627 0.886275 0.952941 1" />
+          <color rgba="0.933333 0.933333 0.933333 1" />
         </material>
       </visual>
@@ -120,16 +120,16 @@
     <link name="left_ankle_yaw">
       <inertial>
-        <origin xyz="-0.00320174 -1.74867e-05 -0.180446" rpy="0 0 0" />
-        <mass value="1.382" />
-        <inertia ixx="0.00852579" ixy="-2.28586e-06" ixz="7.09637e-05" iyy="0.00864443" iyz="-9.78554e-07" izz="0.00102056" />
+        <origin xyz="-0.00304992 0.00150525 -0.18535" rpy="0 0 0" />
+        <mass value="1.43174" />
+        <inertia ixx="0.00763083" ixy="3.0411e-06" ixz="0.000159775" iyy="0.00768647" iyz="-2.6083e-05" izz="0.00115305" />
       </inertial>
       <!-- Part left_ankle_yaw_parts -->
       <visual>
-        <origin xyz="-0.00320174 -1.74867e-05 -0.180446" rpy="-0 0 -0" />
+        <origin xyz="-0.00304992 0.00150525 -0.18535" rpy="-0 0 -0" />
         <geometry>
           <mesh filename="${mesh_root}/left_ankle_yaw_visual.stl" />
         </geometry>
         <material name="left_ankle_yaw_parts_material">
-          <color rgba="0.768627 0.886275 0.952941 1" />
+          <color rgba="0.933333 0.933333 0.933333 1" />
         </material>
       </visual>
@@ -138,16 +138,16 @@
     <link name="left_ankle_pitch">
       <inertial>
-        <origin xyz="0 0.018659 -0" rpy="0 0 0" />
-        <mass value="0.136941" />
-        <inertia ixx="7.39195e-05" ixy="-0" ixz="0" iyy="3.54787e-05" iyz="-0" izz="7.28807e-05" />
+        <origin xyz="-0.00384209 0.0297371 3.1356e-08" rpy="0 0 0" />
+        <mass value="0.184118" />
+        <inertia ixx="9.75514e-05" ixy="-1.6796e-05" ixz="-4.2e-11" iyy="7.7573e-05" iyz="1.44e-10" izz="0.00013275" />
       </inertial>
       <!-- Part left_ankle_pitch_parts -->
       <visual>
-        <origin xyz="0 0.018659 -0" rpy="1.5708 0 0" />
+        <origin xyz="-0.00384209 0.0297371 3.1356e-08" rpy="1.5708 -0 -0" />
         <geometry>
           <mesh filename="${mesh_root}/left_ankle_pitch_visual.stl" />
         </geometry>
         <material name="left_ankle_pitch_parts_material">
-          <color rgba="0.980392 0.713725 0.00392157 1" />
+          <color rgba="0.933333 0.933333 0.933333 1" />
         </material>
       </visual>
@@ -156,11 +156,11 @@
     <link name="left_foot">
       <inertial>
-        <origin xyz="0.00117111 0.0221805 0.0383837" rpy="0 0 0" />
-        <mass value="1.18451" />
-        <inertia ixx="0.00350801" ixy="-6.2179e-06" ixz="-0.000109961" iyy="0.00312661" iyz="-0.000370785" izz="0.00128477" />
+        <origin xyz="0.00124938 0.0227876 0.0398042" rpy="0 0 0" />
+        <mass value="1.20654" />
+        <inertia ixx="0.00367026" ixy="-9.09996e-06" ixz="-0.000117811" iyy="0.00327589" iyz="-0.000424612" izz="0.00132106" />
       </inertial>
       <!-- Part left_foot_parts -->
       <collision>
-        <origin xyz="0 0.05 0.015" rpy="1.5708 -0 0" />
+        <origin xyz="0 0.08 0.015" rpy="1.5708 0 0" />
         <geometry>
           <box size="0.065 0.12 0.03" />
@@ -168,5 +168,5 @@
       </collision>
       <collision>
-        <origin xyz="0 0.04 0.11" rpy="1.91986 -0 0" />
+        <origin xyz="0 0.07 0.11" rpy="1.91986 0 0" />
         <geometry>
           <box size="0.07 0.05 0.03" />
@@ -174,10 +174,10 @@
       </collision>
       <visual>
-        <origin xyz="0.00117111 0.0221805 0.0383837" rpy="1.5708 -1.5708 0" />
+        <origin xyz="0.00124938 0.0227876 0.0398042" rpy="1.5708 -1.5708 0" />
         <geometry>
           <mesh filename="${mesh_root}/left_foot_visual.stl" />
         </geometry>
         <material name="left_foot_parts_material">
-          <color rgba="0.231373 0.380392 0.705882 1" />
+          <color rgba="0.933333 0.933333 0.933333 1" />
         </material>
       </visual>
@@ -185,5 +185,5 @@
     <!-- Joint from left_ankle_pitch to left_foot -->
     <joint name="left_ankle_roll" type="revolute">
-      <origin xyz="0 0.04 -0" rpy="-0 1.5708 0" />
+      <origin xyz="-0 0.04 0" rpy="0 1.5708 0" />
       <parent link="left_ankle_pitch" />
       <child link="left_foot" />
@@ -194,54 +194,54 @@
     <!-- Joint from left_ankle_yaw to left_ankle_pitch -->
     <joint name="left_ankle_pitch" type="revolute">
-      <origin xyz="-0 -0 -0.37" rpy="-1.5708 -0 0" />
+      <origin xyz="0.01 -0 -0.34" rpy="-1.5708 0 -0" />
       <parent link="left_ankle_yaw" />
       <child link="left_ankle_pitch" />
       <axis xyz="0 0 1" />
-      <limit effort="27.0" velocity="100" lower="-0.785398" upper="0.785398" />
+      <limit effort="14.0" velocity="100" lower="-0.523599" upper="0.872665" />
       <joint_properties friction="0.1" />
     </joint>
     <!-- Joint from left_knee_pitch to left_ankle_yaw -->
     <joint name="left_ankle_yaw" type="revolute">
-      <origin xyz="-0.015 0 0" rpy="1.5708 -0 -0" />
+      <origin xyz="-0.015 0 0" rpy="1.5708 0 -0" />
       <parent link="left_knee_pitch" />
       <child link="left_ankle_yaw" />
       <axis xyz="0 0 1" />
-      <limit effort="27.0" velocity="100" lower="-0.785398" upper="0.785398" />
+      <limit effort="14.0" velocity="100" lower="-0.785398" upper="0.785398" />
       <joint_properties friction="0.1" />
     </joint>
     <!-- Joint from left_hip_yaw to left_knee_pitch -->
     <joint name="left_knee_pitch" type="revolute">
-      <origin xyz="-0.01 -0 -0.33" rpy="-1.5708 0 0" />
+      <origin xyz="-0.01 0 -0.33" rpy="-1.5708 0 0" />
       <parent link="left_hip_yaw" />
       <child link="left_knee_pitch" />
       <axis xyz="0 0 1" />
-      <limit effort="97.0" velocity="100" lower="0" upper="2.0944" />
+      <limit effort="36.0" velocity="100" lower="0" upper="2.35619" />
       <joint_properties friction="0.1" />
     </joint>
     <!-- Joint from left_hip_roll to left_hip_yaw -->
     <joint name="left_hip_yaw" type="revolute">
-      <origin xyz="0 -0.0068404 -0.0187939" rpy="-0 -1.22173 1.5708" />
+      <origin xyz="0 -0.0068404 -0.0187939" rpy="0 -1.22173 1.5708" />
       <parent link="left_hip_roll" />
       <child link="left_hip_yaw" />
       <axis xyz="0 0 1" />
-      <limit effort="97.0" velocity="100" lower="-1.5708" upper="1.5708" />
+      <limit effort="17.0" velocity="100" lower="-1.5708" upper="1.5708" />
       <joint_properties friction="0.1" />
     </joint>
     <!-- Joint from left_hip_pitch to left_hip_roll -->
     <joint name="left_hip_roll" type="revolute">
-      <origin xyz="0 0 0" rpy="1.91986 1.39626 1.5708" />
+      <origin xyz="-0 0 -0" rpy="1.91986 1.39626 1.5708" />
       <parent link="left_hip_pitch" />
       <child link="left_hip_roll" />
       <axis xyz="0 0 1" />
-      <limit effort="97.0" velocity="100" lower="-0.349066" upper="1.5708" />
+      <limit effort="36.0" velocity="100" lower="-0.349066" upper="1.5708" />
       <joint_properties friction="0.1" />
     </joint>
     <!-- Joint from pelvis to left_hip_pitch -->
     <joint name="left_hip_pitch" type="revolute">
-      <origin xyz="0.02 0.07 0" rpy="-1.74533 -0 0" />
+      <origin xyz="0.02 0.07 0" rpy="-1.74533 0 0" />
       <parent link="pelvis" />
       <child link="left_hip_pitch" />
       <axis xyz="0 0 1" />
-      <limit effort="97.0" velocity="100" lower="-2.35619" upper="0.785398" />
+      <limit effort="36.0" velocity="100" lower="-2.35619" upper="0.785398" />
       <joint_properties friction="0.1" />
     </joint>
@@ -249,16 +249,16 @@
     <link name="right_hip_pitch">
       <inertial>
-        <origin xyz="-0.0102358 0.00373283 -0.0191788" rpy="0 0 0" />
-        <mass value="0.595116" />
-        <inertia ixx="0.000596331" ixy="5.62188e-05" ixz="0.00011087" iyy="0.000729588" iyz="-4.15218e-05" izz="0.000918618" />
+        <origin xyz="-0.0114771 0.00418737 -0.0187964" rpy="0 0 0" />
+        <mass value="0.619423" />
+        <inertia ixx="0.000652275" ixy="5.37438e-05" ixz="0.000118863" iyy="0.000778995" iyz="-4.4778e-05" izz="0.000986036" />
       </inertial>
       <!-- Part right_hip_pitch_parts -->
       <visual>
-        <origin xyz="-0.0102358 0.00373283 -0.0191788" rpy="1.39626 0 0" />
+        <origin xyz="-0.0114771 0.00418737 -0.0187964" rpy="1.39626 0 -0" />
         <geometry>
           <mesh filename="${mesh_root}/right_hip_pitch_visual.stl" />
         </geometry>
         <material name="right_hip_pitch_parts_material">
-          <color rgba="0.498039 0.498039 0.498039 1" />
+          <color rgba="0.933333 0.933333 0.933333 1" />
         </material>
       </visual>
@@ -267,11 +267,11 @@
     <link name="right_hip_roll">
       <inertial>
-        <origin xyz="-6.2482e-08 0.055907 -0.0657733" rpy="0 0 0" />
-        <mass value="1.12092" />
-        <inertia ixx="0.00291118" ixy="1.0985e-08" ixz="1.48e-08" iyy="0.001481" iyz="-0.000661064" izz="0.00295542" />
+        <origin xyz="-1.13349e-07 0.0525083 -0.0652488" rpy="0 0 0" />
+        <mass value="1.30368" />
+        <inertia ixx="0.0036888" ixy="3.8e-10" ixz="8.521e-09" iyy="0.00199598" iyz="-0.000913166" izz="0.0035815" />
       </inertial>
       <!-- Part right_hip_roll_parts -->
       <collision>
-        <origin xyz="0 0.181098 -0.0871979" rpy="1.22173 -0 0" />
+        <origin xyz="-0 0.181098 -0.0871979" rpy="1.22173 0 0" />
         <geometry>
           <cylinder length="0.15" radius="0.05" />
@@ -279,10 +279,10 @@
       </collision>
       <visual>
-        <origin xyz="-6.2482e-08 0.055907 -0.0657733" rpy="0 -1.22173 1.5708" />
+        <origin xyz="-1.13349e-07 0.0525083 -0.0652488" rpy="0 -1.22173 1.5708" />
         <geometry>
           <mesh filename="${mesh_root}/right_hip_roll_visual.stl" />
         </geometry>
         <material name="right_hip_roll_parts_material">
-          <color rgba="0.647059 0.647059 0.647059 1" />
+          <color rgba="0.933333 0.933333 0.933333 1" />
         </material>
       </visual>
@@ -291,16 +291,16 @@
     <link name="right_hip_yaw">
       <inertial>
-        <origin xyz="-0.00141347 3.75107e-05 -0.232605" rpy="0 0 0" />
-        <mass value="2.10215" />
-        <inertia ixx="0.0106161" ixy="-2.40585e-06" ixz="-0.00036457" iyy="0.0108723" iyz="-8.35769e-07" izz="0.00262072" />
+        <origin xyz="0.00130421 2.35733e-05 -0.237299" rpy="0 0 0" />
+        <mass value="2.08959" />
+        <inertia ixx="0.0116206" ixy="-1.08279e-06" ixz="-0.000458016" iyy="0.0118687" iyz="-3.03522e-07" izz="0.00261696" />
       </inertial>
       <!-- Part right_hip_yaw_parts -->
       <visual>
-        <origin xyz="-0.00141347 3.75107e-05 -0.232605" rpy="-0 -0 0" />
+        <origin xyz="0.00130421 2.35733e-05 -0.237299" rpy="0 0 0" />
         <geometry>
           <mesh filename="${mesh_root}/right_hip_yaw_visual.stl" />
         </geometry>
         <material name="right_hip_yaw_parts_material">
-          <color rgba="0.917647 0.917647 0.917647 1" />
+          <color rgba="0.933333 0.933333 0.933333 1" />
         </material>
       </visual>
@@ -309,11 +309,11 @@
     <link name="right_knee_pitch">
       <inertial>
-        <origin xyz="-0.00532006 0.0299356 -3.8479e-06" rpy="0 0 0" />
-        <mass value="0.389417" />
-        <inertia ixx="0.000727366" ixy="4.24746e-05" ixz="2.14178e-06" iyy="0.000543208" iyz="3.25082e-07" izz="0.000490239" />
+        <origin xyz="-0.0048642 0.0372186 0.000224747" rpy="0 0 0" />
+        <mass value="0.435358" />
+        <inertia ixx="0.000913266" ixy="6.65739e-05" ixz="2.14089e-07" iyy="0.000625521" iyz="-1.04876e-06" izz="0.00071467" />
       </inertial>
       <!-- Part right_knee_pitch_parts -->
       <collision>
-        <origin xyz="-0.01 0.17 -0" rpy="1.5708 1.5708 0" />
+        <origin xyz="-0.01 0.17 0" rpy="1.5708 1.5708 0" />
         <geometry>
           <cylinder length="0.16" radius="0.045" />
@@ -321,10 +321,10 @@
       </collision>
       <visual>
-        <origin xyz="-0.00532006 0.0299356 -3.8479e-06" rpy="1.5708 0 -0" />
+        <origin xyz="-0.0048642 0.0372186 0.000224747" rpy="1.5708 -0 0" />
         <geometry>
           <mesh filename="${mesh_root}/right_knee_pitch_visual.stl" />
         </geometry>
         <material name="right_knee_pitch_parts_material">
-          <color rgba="0.768627 0.886275 0.952941 1" />
+          <color rgba="0.933333 0.933333 0.933333 1" />
         </material>
       </visual>
@@ -333,16 +333,16 @@
     <link name="right_ankle_yaw">
       <inertial>
-        <origin xyz="-0.00320161 1.76517e-05 -0.180446" rpy="0 0 0" />
-        <mass value="1.382" />
-        <inertia ixx="0.00852573" ixy="2.29155e-06" ixz="7.09582e-05" iyy="0.00864437" iyz="9.75164e-07" izz="0.00102056" />
+        <origin xyz="-0.00304909 -0.00150539 -0.185348" rpy="0 0 0" />
+        <mass value="1.43169" />
+        <inertia ixx="0.00763064" ixy="-3.05072e-06" ixz="0.000159784" iyy="0.00768622" iyz="2.60897e-05" izz="0.00115301" />
       </inertial>
       <!-- Part right_ankle_yaw_parts -->
       <visual>
-        <origin xyz="-0.00320161 1.76517e-05 -0.180446" rpy="-0 -0 -0" />
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
File: robots/lite_biped/urdf/lite_biped.urdf (robot description, URDF)
Before this commit: robot lite_biped, 15 links, 14 joints
Joints:
- joint left_ankle_pitch: limit lower=-0.523599 upper=0.872665 effort=27.0 velocity=100 -> lower=-0.523599 upper=0.872665 effort=14.0 velocity=100
- joint left_ankle_yaw: limit lower=-0.785398 upper=0.785398 effort=27.0 velocity=100 -> lower=-0.785398 upper=0.785398 effort=14.0 velocity=100
- joint left_hip_pitch: limit lower=-2.35619 upper=0.785398 effort=97.0 velocity=100 -> lower=-2.35619 upper=0.785398 effort=36.0 velocity=100
- joint left_hip_roll: limit lower=-0.349066 upper=1.5708 effort=97.0 velocity=100 -> lower=-0.349066 upper=1.5708 effort=36.0 velocity=100
- joint left_hip_yaw: limit lower=-1.5708 upper=1.5708 effort=97.0 velocity=100 -> lower=-1.5708 upper=1.5708 effort=17.0 velocity=100
- joint left_knee_pitch: limit lower=0 upper=2.35619 effort=97.0 velocity=100 -> lower=0 upper=2.35619 effort=36.0 velocity=100
- joint right_ankle_pitch: limit lower=-0.523599 upper=0.872665 effort=27.0 velocity=100 -> lower=-0.523599 upper=0.872665 effort=14.0 velocity=100
- joint right_ankle_yaw: limit lower=-0.785398 upper=0.785398 effort=27.0 velocity=100 -> lower=-0.785398 upper=0.785398 effort=14.0 velocity=100
- joint right_hip_pitch: limit lower=-2.35619 upper=0.785398 effort=97.0 velocity=100 -> lower=-2.35619 upper=0.785398 effort=36.0 velocity=100
- joint right_hip_roll: limit lower=-1.5708 upper=0.349066 effort=97.0 velocity=100 -> lower=-1.5708 upper=0.349066 effort=36.0 velocity=100
- joint right_hip_yaw: limit lower=-1.5708 upper=1.5708 effort=97.0 velocity=100 -> lower=-1.5708 upper=1.5708 effort=17.0 velocity=100
- joint right_knee_pitch: limit lower=0 upper=2.35619 effort=97.0 velocity=100 -> lower=0 upper=2.35619 effort=36.0 velocity=100
