Commit message: Add lite_pro variant; update lite from CAD; verify actuator joint params
Add the lite_pro full-body humanoid and align actuator-derived joint
parameters across the full-body variants against the actuator manuals
(Actuator-Manuals/). Convention: effort_limit = the manual's peak torque;
armature/friction_loss are sysid priors (not in the manuals).

lite_pro (new; 74 DoF; root pelvis; model-only):
- Generated from the Onshape "Humanoid Pro" assembly via the offline
  --convert path; colliders reused from lite (pelvis.scad -> waist.scad to
  match the new root part).
- Arms Robstride: shoulder_pitch RS02 (17 Nm); shoulder roll/yaw + elbow
  RS00 (14); wrist RS05 (5.5). Legs+waist DM: hip pitch/roll + knee +
  waist_yaw DM-J6248P (97); hip_yaw + ankle yaw/pitch + waist roll/pitch
  DM-J4340P (40); ankle_roll RS05 (5.5). Neck Sitodrive TA40 100:1 (9);
  fingers placeholder.

lite (regenerated from updated export):
- Waist simplified 3-DoF -> 1-DoF (waist_yaw only); now 72 DoF.
- Legs on Robstride: hip/knee RS06 (36), hip_yaw RS02 (17), ankle
  yaw/pitch RS00 (14), ankle_roll RS05 (5.5).

lite_biped: legs aligned to the same Robstride mapping (was stale 97 Nm).

Register lite_pro in CMakeLists; update the README variants table.
All 1376 tests pass.

Co-Authored-By: Claude Opus 4.8 (1M context) <noreply@anthropic.com>
Claude-Session: https://claude.ai/code/session_01KXLFn7xhCYz59LiUie9B9k

File: robots/lite_biped/xacro/lite_biped.description.xacro (robot description, xacro)
@@ -192,5 +192,5 @@
       <child link="left_ankle_pitch" />
       <axis xyz="0 0 1" />
-      <limit effort="27.0" velocity="100" lower="-0.523599" upper="0.872665" />
+      <limit effort="14.0" velocity="100" lower="-0.523599" upper="0.872665" />
       <joint_properties friction="0.1" />
     </joint>
@@ -201,5 +201,5 @@
       <child link="left_ankle_yaw" />
       <axis xyz="0 0 1" />
-      <limit effort="27.0" velocity="100" lower="-0.785398" upper="0.785398" />
+      <limit effort="14.0" velocity="100" lower="-0.785398" upper="0.785398" />
       <joint_properties friction="0.1" />
     </joint>
@@ -210,5 +210,5 @@
       <child link="left_knee_pitch" />
       <axis xyz="0 0 1" />
-      <limit effort="97.0" velocity="100" lower="0" upper="2.35619" />
+      <limit effort="36.0" velocity="100" lower="0" upper="2.35619" />
       <joint_properties friction="0.1" />
     </joint>
@@ -219,5 +219,5 @@
       <child link="left_hip_yaw" />
       <axis xyz="0 0 1" />
-      <limit effort="97.0" velocity="100" lower="-1.5708" upper="1.5708" />
+      <limit effort="17.0" velocity="100" lower="-1.5708" upper="1.5708" />
       <joint_properties friction="0.1" />
     </joint>
@@ -228,5 +228,5 @@
       <child link="left_hip_roll" />
       <axis xyz="0 0 1" />
-      <limit effort="97.0" velocity="100" lower="-0.349066" upper="1.5708" />
+      <limit effort="36.0" velocity="100" lower="-0.349066" upper="1.5708" />
       <joint_properties friction="0.1" />
     </joint>
@@ -237,5 +237,5 @@
       <child link="left_hip_pitch" />
       <axis xyz="0 0 1" />
-      <limit effort="97.0" velocity="100" lower="-2.35619" upper="0.785398" />
+      <limit effort="36.0" velocity="100" lower="-2.35619" upper="0.785398" />
       <joint_properties friction="0.1" />
     </joint>
@@ -405,5 +405,5 @@
       <child link="right_ankle_pitch" />
       <axis xyz="0 0 1" />
-      <limit effort="27.0" velocity="100" lower="-0.523599" upper="0.872665" />
+      <limit effort="14.0" velocity="100" lower="-0.523599" upper="0.872665" />
       <joint_properties friction="0.1" />
     </joint>
@@ -414,5 +414,5 @@
       <child link="right_ankle_yaw" />
       <axis xyz="0 0 1" />
-      <limit effort="27.0" velocity="100" lower="-0.785398" upper="0.785398" />
+      <limit effort="14.0" velocity="100" lower="-0.785398" upper="0.785398" />
       <joint_properties friction="0.1" />
     </joint>
@@ -423,5 +423,5 @@
       <child link="right_knee_pitch" />
       <axis xyz="0 0 1" />
-      <limit effort="97.0" velocity="100" lower="0" upper="2.35619" />
+      <limit effort="36.0" velocity="100" lower="0" upper="2.35619" />
       <joint_properties friction="0.1" />
     </joint>
@@ -432,5 +432,5 @@
       <child link="right_hip_yaw" />
       <axis xyz="0 0 1" />
-      <limit effort="97.0" velocity="100" lower="-1.5708" upper="1.5708" />
+      <limit effort="17.0" velocity="100" lower="-1.5708" upper="1.5708" />
       <joint_properties friction="0.1" />
     </joint>
@@ -441,5 +441,5 @@
       <child link="right_hip_roll" />
       <axis xyz="0 0 1" />
-      <limit effort="97.0" velocity="100" lower="-1.5708" upper="0.349066" />
+      <limit effort="36.0" velocity="100" lower="-1.5708" upper="0.349066" />
       <joint_properties friction="0.1" />
     </joint>
@@ -450,5 +450,5 @@
       <child link="right_hip_pitch" />
       <axis xyz="0 0 1" />
-      <limit effort="97.0" velocity="100" lower="-2.35619" upper="0.785398" />
+      <limit effort="36.0" velocity="100" lower="-2.35619" upper="0.785398" />
       <joint_properties friction="0.1" />
     </joint>
