Commit message: refactor: directory structure

File: robots/lite/urdf/lite.urdf (robot description, URDF)
Before this commit: robot lite, 75 links, 74 joints
Links:
- link chest: geometry collision box size=0.08 0.1 0.18; visual mesh filename=../meshes/visual/chest_visual.stl
- link head: geometry collision cylinder length=0.03 radius=0.09; visual mesh filename=../meshes/visual/head_visual.stl
- link left_ankle_pitch: geometry visual mesh filename=../meshes/visual/left_ankle_pitch_visual.stl
- link left_ankle_yaw: geometry visual mesh filename=../meshes/visual/left_ankle_yaw_visual.stl
- link left_elbow_pitch: geometry visual mesh filename=../meshes/visual/left_elbow_pitch_visual.stl
- link left_finger1_j1: geometry visual mesh filename=../meshes/visual/left_finger1_j1_visual.stl
- link left_finger1_j2: geometry visual mesh filename=../meshes/visual/left_finger1_j2_visual.stl
- link left_finger1_j3: geometry visual mesh filename=../meshes/visual/left_finger1_j3_visual.stl
- link left_finger1_j4: geometry visual mesh filename=../meshes/visual/left_finger1_j4_visual.stl
- link left_finger2_j1: geometry visual mesh filename=../meshes/visual/left_finger2_j1_visual.stl
- link left_finger2_j2: geometry visual mesh filename=../meshes/visual/left_finger2_j2_visual.stl
- link left_finger2_j3: geometry visual mesh filename=../meshes/visual/left_finger2_j3_visual.stl
- link left_finger2_j4: geometry visual mesh filename=../meshes/visual/left_finger2_j4_visual.stl
- link left_finger3_j1: geometry visual mesh filename=../meshes/visual/left_finger3_j1_visual.stl
- link left_finger3_j2: geometry visual mesh filename=../meshes/visual/left_finger3_j2_visual.stl
- link left_finger3_j3: geometry visual mesh filename=../meshes/visual/left_finger3_j3_visual.stl
- link left_finger3_j4: geometry visual mesh filename=../meshes/visual/left_finger3_j4_visual.stl
- link left_finger4_j1: geometry visual mesh filename=../meshes/visual/left_finger4_j1_visual.stl
- link left_finger4_j2: geometry visual mesh filename=../meshes/visual/left_finger4_j2_visual.stl
- link left_finger4_j3: geometry visual mesh filename=../meshes/visual/left_finger4_j3_visual.stl
- link left_finger4_j4: geometry visual mesh filename=../meshes/visual/left_finger4_j4_visual.stl
- link left_finger5_j1: geometry visual mesh filename=../meshes/visual/left_finger5_j1_visual.stl
- link left_finger5_j2: geometry visual mesh filename=../meshes/visual/left_finger5_j2_visual.stl
- link left_finger5_j3: geometry visual mesh filename=../meshes/visual/left_finger5_j3_visual.stl
- link left_finger5_j4: geometry visual mesh filename=../meshes/visual/left_finger5_j4_visual.stl
- link left_foot: geometry collision box size=0.065 0.12 0.03; collision box size=0.07 0.05 0.03
- link left_hand: geometry collision box size=0.1 0.07 0.015; visual mesh filename=../meshes/visual/left_hand_visual.stl
- link left_hip_pitch: geometry visual mesh filename=../meshes/visual/left_hip_pitch_visual.stl
- link left_hip_roll: geometry collision cylinder length=0.15 radius=0.05; visual mesh filename=../meshes/visual/left_hip_roll_visual.stl
- link left_hip_yaw: geometry visual mesh filename=../meshes/visual/left_hip_yaw_visual.stl
- link left_knee_pitch: geometry collision cylinder length=0.16 radius=0.045; visual mesh filename=../meshes/visual/left_knee_pitch_visual.stl
- link left_shoulder_pitch: geometry visual mesh filename=../meshes/visual/left_shoulder_pitch_visual.stl
- link left_shoulder_roll: geometry visual mesh filename=../meshes/visual/left_shoulder_roll_visual.stl
- link left_shoulder_yaw: geometry collision cylinder length=0.08 radius=0.03; visual mesh filename=../meshes/visual/left_shoulder_yaw_visual.stl
- link left_wrist_roll: geometry visual mesh filename=../meshes/visual/left_wrist_roll_visual.stl
- link left_wrist_yaw: geometry collision cylinder length=0.06 radius=0.03; visual mesh filename=../meshes/visual/left_wrist_yaw_visual.stl
- link neck_roll: geometry visual mesh filename=../meshes/visual/neck_roll_visual.stl
- link neck_yaw: geometry visual mesh filename=../meshes/visual/neck_yaw_visual.stl
- link pelvis: geometry collision cylinder length=0.16 radius=0.05; visual mesh filename=../meshes/visual/pelvis_visual.stl
- link right_ankle_pitch: geometry visual mesh filename=../meshes/visual/right_ankle_pitch_visual.stl
- link right_ankle_yaw: geometry visual mesh filename=../meshes/visual/right_ankle_yaw_visual.stl
- link right_elbow_pitch: geometry visual mesh filename=../meshes/visual/right_elbow_pitch_visual.stl
- link right_finger1_j1: geometry visual mesh filename=../meshes/visual/right_finger1_j1_visual.stl
- link right_finger1_j2: geometry visual mesh filename=../meshes/visual/right_finger1_j2_visual.stl
- link right_finger1_j3: geometry visual mesh filename=../meshes/visual/right_finger1_j3_visual.stl
- link right_finger1_j4: geometry visual mesh filename=../meshes/visual/right_finger1_j4_visual.stl
- link right_finger2_j1: geometry visual mesh filename=../meshes/visual/right_finger2_j1_visual.stl
- link right_finger2_j2: geometry visual mesh filename=../meshes/visual/right_finger2_j2_visual.stl
- link right_finger2_j3: geometry visual mesh filename=../meshes/visual/right_finger2_j3_visual.stl
- link right_finger2_j4: geometry visual mesh filename=../meshes/visual/right_finger2_j4_visual.stl
- link right_finger3_j1: geometry visual mesh filename=../meshes/visual/right_finger3_j1_visual.stl
- link right_finger3_j2: geometry visual mesh filename=../meshes/visual/right_finger3_j2_visual.stl
- link right_finger3_j3: geometry visual mesh filename=../meshes/visual/right_finger3_j3_visual.stl
- link right_finger3_j4: geometry visual mesh filename=../meshes/visual/right_finger3_j4_visual.stl
- link right_finger4_j1: geometry visual mesh filename=../meshes/visual/right_finger4_j1_visual.stl
- link right_finger4_j2: geometry visual mesh filename=../meshes/visual/right_finger4_j2_visual.stl
- link right_finger4_j3: geometry visual mesh filename=../meshes/visual/right_finger4_j3_visual.stl
- link right_finger4_j4: geometry visual mesh filename=../meshes/visual/right_finger4_j4_visual.stl
- link right_finger5_j1: geometry visual mesh filename=../meshes/visual/right_finger5_j1_visual.stl
- link right_finger5_j2: geometry visual mesh filename=../meshes/visual/right_finger5_j2_visual.stl
- link right_finger5_j3: geometry visual mesh filename=../meshes/visual/right_finger5_j3_visual.stl
- link right_finger5_j4: geometry visual mesh filename=../meshes/visual/right_finger5_j4_visual.stl
- link right_foot: geometry collision box size=0.065 0.12 0.03; collision box size=0.07 0.05 0.03
- link right_hand: geometry collision box size=0.1 0.07 0.015; visual mesh filename=../meshes/visual/right_hand_visual.stl
- link right_hip_pitch: geometry visual mesh filename=../meshes/visual/right_hip_pitch_visual.stl
- link right_hip_roll: geometry collision cylinder length=0.15 radius=0.05; visual mesh filename=../meshes/visual/right_hip_roll_visual.stl
- link right_hip_yaw: geometry visual mesh filename=../meshes/visual/right_hip_yaw_visual.stl
- link right_knee_pitch: geometry collision cylinder length=0.16 radius=0.045; visual mesh filename=../meshes/visual/right_knee_pitch_visual.stl
- link right_shoulder_pitch: geometry visual mesh filename=../meshes/visual/right_shoulder_pitch_visual.stl
- link right_shoulder_roll: geometry visual mesh filename=../meshes/visual/right_shoulder_roll_visual.stl
- link right_shoulder_yaw: geometry collision cylinder length=0.08 radius=0.03; visual mesh filename=../meshes/visual/right_shoulder_yaw_visual.stl
- link right_wrist_roll: geometry visual mesh filename=../meshes/visual/right_wrist_roll_visual.stl
- link right_wrist_yaw: geometry collision cylinder length=0.06 radius=0.03; visual mesh filename=../meshes/visual/right_wrist_yaw_visual.stl
- link waist_pitch: geometry visual mesh filename=../meshes/visual/waist_pitch_visual.stl
- link waist_yaw: geometry visual mesh filename=../meshes/visual/waist_yaw_visual.stl
Joints:
- joint left_ankle_pitch: limit lower=-0.785398 upper=0.785398 effort=100 velocity=100 -> lower=-0.785398 upper=0.785398 effort=27.0 velocity=100
- joint left_ankle_roll: limit lower=-0.349066 upper=0.349066 effort=100 velocity=100 -> lower=-0.349066 upper=0.349066 effort=5.5 velocity=100
- joint left_ankle_yaw: limit lower=-0.785398 upper=0.785398 effort=100 velocity=100 -> lower=-0.785398 upper=0.785398 effort=27.0 velocity=100
- joint left_elbow_pitch: limit lower=-2.35619 upper=0 effort=100 velocity=100 -> lower=-2.35619 upper=0 effort=14.0 velocity=100
- joint left_finger1_j1: limit lower=-1.5708 upper=-0 effort=100 velocity=100 -> lower=-1.5708 upper=-0 effort=10 velocity=100
- joint left_finger1_j2: limit lower=-0.349066 upper=0.349066 effort=100 velocity=100 -> lower=-0.349066 upper=0.349066 effort=10 velocity=100
- joint left_finger1_j3: limit lower=-1.91986 upper=0.0872665 effort=100 velocity=100 -> lower=-1.91986 upper=0.0872665 effort=10 velocity=100
- joint left_finger1_j4: limit lower=-1.5708 upper=0.0872665 effort=100 velocity=100 -> lower=-1.5708 upper=0.0872665 effort=10 velocity=100
- joint left_finger2_j1: limit lower=-1.91986 upper=0.0872665 effort=100 velocity=100 -> lower=-1.91986 upper=0.0872665 effort=10 velocity=100
- joint left_finger2_j2: limit lower=-0.349066 upper=0.349066 effort=100 velocity=100 -> lower=-0.349066 upper=0.349066 effort=10 velocity=100
- joint left_finger2_j3: limit lower=-1.91986 upper=0.0872665 effort=100 velocity=100 -> lower=-1.91986 upper=0.0872665 effort=10 velocity=100
- joint left_finger2_j4: limit lower=-1.5708 upper=0.0872665 effort=100 velocity=100 -> lower=-1.5708 upper=0.0872665 effort=10 velocity=100
- joint left_finger3_j1: limit lower=-1.91986 upper=0.0872665 effort=100 velocity=100 -> lower=-1.91986 upper=0.0872665 effort=10 velocity=100
- joint left_finger3_j2: limit lower=-0.349066 upper=0.349066 effort=100 velocity=100 -> lower=-0.349066 upper=0.349066 effort=10 velocity=100
- joint left_finger3_j3: limit lower=-1.91986 upper=0.0872665 effort=100 velocity=100 -> lower=-1.91986 upper=0.0872665 effort=10 velocity=100
- joint left_finger3_j4: limit lower=-1.5708 upper=0.0872665 effort=100 velocity=100 -> lower=-1.5708 upper=0.0872665 effort=10 velocity=100
- joint left_finger4_j1: limit lower=-1.91986 upper=0.0872665 effort=100 velocity=100 -> lower=-1.91986 upper=0.0872665 effort=10 velocity=100
- joint left_finger4_j2: limit lower=-0.349066 upper=0.349066 effort=100 velocity=100 -> lower=-0.349066 upper=0.349066 effort=10 velocity=100
- joint left_finger4_j3: limit lower=-1.91986 upper=0.0872665 effort=100 velocity=100 -> lower=-1.91986 upper=0.0872665 effort=10 velocity=100
- joint left_finger4_j4: limit lower=-1.5708 upper=0.0872665 effort=100 velocity=100 -> lower=-1.5708 upper=0.0872665 effort=10 velocity=100
- joint left_finger5_j1: limit lower=-1.91986 upper=0.0872665 effort=100 velocity=100 -> lower=-1.91986 upper=0.0872665 effort=10 velocity=100
- joint left_finger5_j2: limit lower=-0.349066 upper=0.349066 effort=100 velocity=100 -> lower=-0.349066 upper=0.349066 effort=10 velocity=100
- joint left_finger5_j3: limit lower=-1.91986 upper=0.0872665 effort=100 velocity=100 -> lower=-1.91986 upper=0.0872665 effort=10 velocity=100
- joint left_finger5_j4: limit lower=-1.5708 upper=0.0872665 effort=100 velocity=100 -> lower=-1.5708 upper=0.0872665 effort=10 velocity=100
- joint left_hip_pitch: limit lower=-2.35619 upper=0.785398 effort=100 velocity=100 -> lower=-2.35619 upper=0.785398 effort=97.0 velocity=100
- joint left_hip_roll: limit lower=-0.349066 upper=1.5708 effort=100 velocity=100 -> lower=-0.349066 upper=1.5708 effort=97.0 velocity=100
- joint left_hip_yaw: limit lower=-1.5708 upper=1.5708 effort=100 velocity=100 -> lower=-1.5708 upper=1.5708 effort=97.0 velocity=100
- joint left_knee_pitch: limit lower=0 upper=2.0944 effort=100 velocity=100 -> lower=0 upper=2.0944 effort=97.0 velocity=100
- joint left_shoulder_pitch: limit lower=-3.14159 upper=0.785398 effort=100 velocity=100 -> lower=-3.14159 upper=0.785398 effort=17.0 velocity=100
- joint left_shoulder_roll: limit lower=-1.5708 upper=1.91986 effort=100 velocity=100 -> lower=-1.5708 upper=1.91986 effort=14.0 velocity=100
- joint left_shoulder_yaw: limit lower=-1.5708 upper=1.5708 effort=100 velocity=100 -> lower=-1.5708 upper=1.5708 effort=14.0 velocity=100
- joint left_wrist_pitch: limit lower=-0.785398 upper=0.785398 effort=100 velocity=100 -> lower=-0.785398 upper=0.785398 effort=5.5 velocity=100
- joint left_wrist_roll: limit lower=-0.698132 upper=0.698132 effort=100 velocity=100 -> lower=-0.698132 upper=0.698132 effort=5.5 velocity=100
- joint left_wrist_yaw: limit lower=-1.5708 upper=1.5708 effort=100 velocity=100 -> lower=-1.5708 upper=1.5708 effort=5.5 velocity=100
- joint neck_pitch: limit lower=-0.523599 upper=0.523599 effort=100 velocity=100 -> lower=-0.523599 upper=0.523599 effort=10 velocity=100
- joint neck_roll: limit lower=-0.523599 upper=0.523599 effort=100 velocity=100 -> lower=-0.523599 upper=0.523599 effort=10 velocity=100
- joint neck_yaw: limit lower=-0.785398 upper=0.785398 effort=100 velocity=100 -> lower=-0.785398 upper=0.785398 effort=10 velocity=100
- joint right_ankle_pitch: limit lower=-0.785398 upper=0.785398 effort=100 velocity=100 -> lower=-0.785398 upper=0.785398 effort=27.0 velocity=100
- joint right_ankle_roll: limit lower=-0.349066 upper=0.349066 effort=100 velocity=100 -> lower=-0.349066 upper=0.349066 effort=5.5 velocity=100
- joint right_ankle_yaw: limit lower=-0.785398 upper=0.785398 effort=100 velocity=100 -> lower=-0.785398 upper=0.785398 effort=27.0 velocity=100
- joint right_elbow_pitch: limit lower=-2.35619 upper=0 effort=100 velocity=100 -> lower=-2.35619 upper=0 effort=14.0 velocity=100
- joint right_finger1_j1: limit lower=0 upper=1.5708 effort=100 velocity=100 -> lower=0 upper=1.5708 effort=10 velocity=100
- joint right_finger1_j2: limit lower=-0.349066 upper=0.349066 effort=100 velocity=100 -> lower=-0.349066 upper=0.349066 effort=10 velocity=100
- joint right_finger1_j3: limit lower=-0.0872665 upper=1.91986 effort=100 velocity=100 -> lower=-0.0872665 upper=1.91986 effort=10 velocity=100
- joint right_finger1_j4: limit lower=-0.0872665 upper=1.5708 effort=100 velocity=100 -> lower=-0.0872665 upper=1.5708 effort=10 velocity=100
- joint right_finger2_j1: limit lower=-0.0872665 upper=1.91986 effort=100 velocity=100 -> lower=-0.0872665 upper=1.91986 effort=10 velocity=100
- joint right_finger2_j2: limit lower=-0.349066 upper=0.349066 effort=100 velocity=100 -> lower=-0.349066 upper=0.349066 effort=10 velocity=100
- joint right_finger2_j3: limit lower=-0.0872665 upper=1.91986 effort=100 velocity=100 -> lower=-0.0872665 upper=1.91986 effort=10 velocity=100
- joint right_finger2_j4: limit lower=-0.0872665 upper=1.5708 effort=100 velocity=100 -> lower=-0.0872665 upper=1.5708 effort=10 velocity=100
- joint right_finger3_j1: limit lower=-0.0872665 upper=1.91986 effort=100 velocity=100 -> lower=-0.0872665 upper=1.91986 effort=10 velocity=100
- joint right_finger3_j2: limit lower=-0.349066 upper=0.349066 effort=100 velocity=100 -> lower=-0.349066 upper=0.349066 effort=10 velocity=100
- joint right_finger3_j3: limit lower=-0.0872665 upper=1.91986 effort=100 velocity=100 -> lower=-0.0872665 upper=1.91986 effort=10 velocity=100
- joint right_finger3_j4: limit lower=-0.0872665 upper=1.5708 effort=100 velocity=100 -> lower=-0.0872665 upper=1.5708 effort=10 velocity=100
- joint right_finger4_j1: limit lower=-0.0872665 upper=1.91986 effort=100 velocity=100 -> lower=-0.0872665 upper=1.91986 effort=10 velocity=100
- joint right_finger4_j2: limit lower=-0.349066 upper=0.349066 effort=100 velocity=100 -> lower=-0.349066 upper=0.349066 effort=10 velocity=100
- joint right_finger4_j3: limit lower=-0.0872665 upper=1.91986 effort=100 velocity=100 -> lower=-0.0872665 upper=1.91986 effort=10 velocity=100
- joint right_finger4_j4: limit lower=-0.0872665 upper=1.5708 effort=100 velocity=100 -> lower=-0.0872665 upper=1.5708 effort=10 velocity=100
- joint right_finger5_j1: limit lower=-0.0872665 upper=1.91986 effort=100 velocity=100 -> lower=-0.0872665 upper=1.91986 effort=10 velocity=100
- joint right_finger5_j2: limit lower=-0.349066 upper=0.349066 effort=100 velocity=100 -> lower=-0.349066 upper=0.349066 effort=10 velocity=100
- joint right_finger5_j3: limit lower=-0.0872665 upper=1.91986 effort=100 velocity=100 -> lower=-0.0872665 upper=1.91986 effort=10 velocity=100
- joint right_finger5_j4: limit lower=-0.0872665 upper=1.5708 effort=100 velocity=100 -> lower=-0.0872665 upper=1.5708 effort=10 velocity=100
- joint right_hip_pitch: limit lower=-2.35619 upper=0.785398 effort=100 velocity=100 -> lower=-2.35619 upper=0.785398 effort=97.0 velocity=100
- joint right_hip_roll: limit lower=-1.5708 upper=0.349066 effort=100 velocity=100 -> lower=-1.5708 upper=0.349066 effort=97.0 velocity=100
- joint right_hip_yaw: limit lower=-1.5708 upper=1.5708 effort=100 velocity=100 -> lower=-1.5708 upper=1.5708 effort=97.0 velocity=100
- joint right_knee_pitch: limit lower=0 upper=2.0944 effort=100 velocity=100 -> lower=0 upper=2.0944 effort=97.0 velocity=100
- joint right_shoulder_pitch: limit lower=-3.14159 upper=0.785398 effort=100 velocity=100 -> lower=-3.14159 upper=0.785398 effort=17.0 velocity=100
- joint right_shoulder_roll: limit lower=-1.91986 upper=1.5708 effort=100 velocity=100 -> lower=-1.91986 upper=1.5708 effort=14.0 velocity=100
- joint right_shoulder_yaw: limit lower=-1.5708 upper=1.5708 effort=100 velocity=100 -> lower=-1.5708 upper=1.5708 effort=14.0 velocity=100
- joint right_wrist_pitch: limit lower=-0.785398 upper=0.785398 effort=100 velocity=100 -> lower=-0.785398 upper=0.785398 effort=5.5 velocity=100
- joint right_wrist_roll: limit lower=-0.698132 upper=0.698132 effort=100 velocity=100 -> lower=-0.698132 upper=0.698132 effort=5.5 velocity=100
- joint right_wrist_yaw: limit lower=-1.5708 upper=1.5708 effort=100 velocity=100 -> lower=-1.5708 upper=1.5708 effort=5.5 velocity=100
- joint waist_pitch: limit lower=-0.785398 upper=1.5708 effort=100 velocity=100 -> lower=-0.785398 upper=1.5708 effort=10 velocity=100
- joint waist_roll: limit lower=-1.0472 upper=1.0472 effort=100 velocity=100 -> lower=-1.0472 upper=1.0472 effort=10 velocity=100
- joint waist_yaw: limit lower=-1.5708 upper=1.5708 effort=100 velocity=100 -> lower=-1.5708 upper=1.5708 effort=10 velocity=100
