Commit message: update: actuator parameters

File: robots/lite/urdf/lite.urdf (robot description, URDF)
Before this commit: robot lite, 73 links, 72 joints
Joints:
- joint neck_pitch: limit lower=-0.698132 upper=0.349066 effort=9.0 velocity=100 -> lower=-0.698132 upper=0.349066 effort=4.8 velocity=100
- joint neck_roll: limit lower=-0.523599 upper=0.523599 effort=9.0 velocity=100 -> lower=-0.523599 upper=0.523599 effort=4.8 velocity=100
- joint neck_yaw: limit lower=-0.785398 upper=0.785398 effort=9.0 velocity=100 -> lower=-0.785398 upper=0.785398 effort=4.8 velocity=100

File: robots/lite/xacro/lite.description.xacro (robot description, xacro)
@@ -2043,5 +2043,5 @@
       <child link="head" />
       <axis xyz="0 0 1" />
-      <limit effort="9.0" velocity="100" lower="-0.698132" upper="0.349066" />
+      <limit effort="4.8" velocity="100" lower="-0.698132" upper="0.349066" />
       <joint_properties friction="0.1" />
     </joint>
@@ -2052,5 +2052,5 @@
       <child link="neck_roll" />
       <axis xyz="0 0 1" />
-      <limit effort="9.0" velocity="100" lower="-0.523599" upper="0.523599" />
+      <limit effort="4.8" velocity="100" lower="-0.523599" upper="0.523599" />
       <joint_properties friction="0.1" />
     </joint>
@@ -2061,5 +2061,5 @@
       <child link="neck_yaw" />
       <axis xyz="0 0 1" />
-      <limit effort="9.0" velocity="100" lower="-0.785398" upper="0.785398" />
+      <limit effort="4.8" velocity="100" lower="-0.785398" upper="0.785398" />
       <joint_properties friction="0.1" />
     </joint>

File: robots/lite_pro/urdf/lite_pro.urdf (robot description, URDF)
Before this commit: robot lite_pro, 75 links, 74 joints
Joints:
- joint left_ankle_pitch: limit lower=-0.523599 upper=0.872665 effort=40.0 velocity=100 -> lower=-0.523599 upper=0.872665 effort=27.0 velocity=100
- joint left_ankle_yaw: limit lower=-0.785398 upper=0.785398 effort=40.0 velocity=100 -> lower=-0.785398 upper=0.785398 effort=27.0 velocity=100
- joint left_hip_yaw: limit lower=-1.5708 upper=1.5708 effort=40.0 velocity=100 -> lower=-1.5708 upper=1.5708 effort=27.0 velocity=100
- joint neck_pitch: limit lower=-0.523599 upper=0.523599 effort=9.0 velocity=100 -> lower=-0.523599 upper=0.523599 effort=4.8 velocity=100
- joint neck_roll: limit lower=-0.523599 upper=0.523599 effort=9.0 velocity=100 -> lower=-0.523599 upper=0.523599 effort=4.8 velocity=100
- joint neck_yaw: limit lower=-0.785398 upper=0.785398 effort=9.0 velocity=100 -> lower=-0.785398 upper=0.785398 effort=4.8 velocity=100
- joint right_ankle_pitch: limit lower=-0.523599 upper=0.872665 effort=40.0 velocity=100 -> lower=-0.523599 upper=0.872665 effort=27.0 velocity=100
- joint right_ankle_yaw: limit lower=-0.785398 upper=0.785398 effort=40.0 velocity=100 -> lower=-0.785398 upper=0.785398 effort=27.0 velocity=100
- joint right_hip_yaw: limit lower=-1.5708 upper=1.5708 effort=40.0 velocity=100 -> lower=-1.5708 upper=1.5708 effort=27.0 velocity=100
- joint waist_pitch: limit lower=-1.5708 upper=0.785398 effort=40.0 velocity=100 -> lower=-1.5708 upper=0.785398 effort=27.0 velocity=100
- joint waist_roll: limit lower=-1.0472 upper=1.0472 effort=40.0 velocity=100 -> lower=-1.0472 upper=1.0472 effort=27.0 velocity=100

File: robots/lite_pro/xacro/lite_pro.description.xacro (robot description, xacro)
@@ -198,5 +198,5 @@
       <child link="left_ankle_pitch" />
       <axis xyz="0 0 1" />
-      <limit effort="40.0" velocity="100" lower="-0.523599" upper="0.872665" />
+      <limit effort="27.0" velocity="100" lower="-0.523599" upper="0.872665" />
       <joint_properties friction="0.1" />
     </joint>
@@ -207,5 +207,5 @@
       <child link="left_ankle_yaw" />
       <axis xyz="0 0 1" />
-      <limit effort="40.0" velocity="100" lower="-0.785398" upper="0.785398" />
+      <limit effort="27.0" velocity="100" lower="-0.785398" upper="0.785398" />
       <joint_properties friction="0.1" />
     </joint>
@@ -225,5 +225,5 @@
       <child link="left_hip_yaw" />
       <axis xyz="0 0 1" />
-      <limit effort="40.0" velocity="100" lower="-1.5708" upper="1.5708" />
+      <limit effort="27.0" velocity="100" lower="-1.5708" upper="1.5708" />
       <joint_properties friction="0.1" />
     </joint>
@@ -411,5 +411,5 @@
       <child link="right_ankle_pitch" />
       <axis xyz="0 0 1" />
-      <limit effort="40.0" velocity="100" lower="-0.523599" upper="0.872665" />
+      <limit effort="27.0" velocity="100" lower="-0.523599" upper="0.872665" />
       <joint_properties friction="0.1" />
     </joint>
@@ -420,5 +420,5 @@
       <child link="right_ankle_yaw" />
       <axis xyz="0 0 1" />
-      <limit effort="40.0" velocity="100" lower="-0.785398" upper="0.785398" />
+      <limit effort="27.0" velocity="100" lower="-0.785398" upper="0.785398" />
       <joint_properties friction="0.1" />
     </joint>
@@ -438,5 +438,5 @@
       <child link="right_hip_yaw" />
       <axis xyz="0 0 1" />
-      <limit effort="40.0" velocity="100" lower="-1.5708" upper="1.5708" />
+      <limit effort="27.0" velocity="100" lower="-1.5708" upper="1.5708" />
       <joint_properties friction="0.1" />
     </joint>
@@ -2079,5 +2079,5 @@
       <child link="head" />
       <axis xyz="0 0 1" />
-      <limit effort="9.0" velocity="100" lower="-0.523599" upper="0.523599" />
+      <limit effort="4.8" velocity="100" lower="-0.523599" upper="0.523599" />
       <joint_properties friction="0.1" />
     </joint>
@@ -2088,5 +2088,5 @@
       <child link="neck_roll" />
       <axis xyz="0 0 1" />
-      <limit effort="9.0" velocity="100" lower="-0.523599" upper="0.523599" />
+      <limit effort="4.8" velocity="100" lower="-0.523599" upper="0.523599" />
       <joint_properties friction="0.1" />
     </joint>
@@ -2097,5 +2097,5 @@
       <child link="neck_yaw" />
       <axis xyz="0 0 1" />
-      <limit effort="9.0" velocity="100" lower="-0.785398" upper="0.785398" />
+      <limit effort="4.8" velocity="100" lower="-0.785398" upper="0.785398" />
       <joint_properties friction="0.1" />
     </joint>
@@ -2106,5 +2106,5 @@
       <child link="chest" />
       <axis xyz="0 0 1" />
-      <limit effort="40.0" velocity="100" lower="-1.5708" upper="0.785398" />
+      <limit effort="27.0" velocity="100" lower="-1.5708" upper="0.785398" />
       <joint_properties friction="0.1" />
     </joint>
@@ -2115,5 +2115,5 @@
       <child link="waist_roll" />
       <axis xyz="0 0 1" />
-      <limit effort="40.0" velocity="100" lower="-1.0472" upper="1.0472" />
+      <limit effort="27.0" velocity="100" lower="-1.0472" upper="1.0472" />
       <joint_properties friction="0.1" />
     </joint>

Commit message: fix: asset colliders

File: robots/lite/urdf/lite.urdf (robot description, URDF)
Before this commit: robot lite, 73 links, 72 joints
Links:
- link left_knee_pitch: geometry collision cylinder length=0.12 radius=0.045; visual mesh filename=../meshes/visual/left_knee_pitch_visual.stl
- link right_knee_pitch: geometry collision cylinder length=0.12 radius=0.045; visual mesh filename=../meshes/visual/right_knee_pitch_visual.stl

File: robots/lite/xacro/lite.description.xacro (robot description, xacro)
@@ -102,7 +102,7 @@
       <!-- Part left_knee_pitch_parts -->
       <collision>
-        <origin xyz="-0.01 0.17 0" rpy="1.5708 1.5708 0" />
-        <geometry>
-          <cylinder length="0.16" radius="0.045" />
+        <origin xyz="-0.015 0.19 0" rpy="1.5708 1.5708 0" />
+        <geometry>
+          <cylinder length="0.12" radius="0.045" />
         </geometry>
       </collision>
@@ -162,5 +162,5 @@
       <!-- Part left_foot_parts -->
       <collision>
-        <origin xyz="0 0.08 0.015" rpy="1.5708 0 0" />
+        <origin xyz="0 0.05 0.015" rpy="1.5708 0 0" />
         <geometry>
           <box size="0.065 0.12 0.03" />
@@ -168,5 +168,5 @@
       </collision>
       <collision>
-        <origin xyz="0 0.07 0.11" rpy="1.91986 0 0" />
+        <origin xyz="0 0.04 0.11" rpy="1.91986 0 0" />
         <geometry>
           <box size="0.07 0.05 0.03" />
@@ -315,7 +315,7 @@
       <!-- Part right_knee_pitch_parts -->
       <collision>
-        <origin xyz="-0.01 0.17 0" rpy="1.5708 1.5708 0" />
-        <geometry>
-          <cylinder length="0.16" radius="0.045" />
+        <origin xyz="-0.015 0.19 0" rpy="1.5708 1.5708 0" />
+        <geometry>
+          <cylinder length="0.12" radius="0.045" />
         </geometry>
       </collision>
@@ -375,5 +375,5 @@
       <!-- Part right_foot_parts -->
       <collision>
-        <origin xyz="0 0.08 0.015" rpy="1.5708 0 -0" />
+        <origin xyz="0 0.05 0.015" rpy="1.5708 0 -0" />
         <geometry>
           <box size="0.065 0.12 0.03" />
@@ -381,5 +381,5 @@
       </collision>
       <collision>
-        <origin xyz="0 0.07 0.11" rpy="1.91986 0 -0" />
+        <origin xyz="0 0.04 0.11" rpy="1.91986 0 -0" />
         <geometry>
           <box size="0.07 0.05 0.03" />

File: robots/lite_biped/urdf/lite_biped.urdf (robot description, URDF)
Before this commit: robot lite_biped, 15 links, 14 joints
Links:
- link left_knee_pitch: geometry collision cylinder length=0.12 radius=0.045; visual mesh filename=../meshes/visual/left_knee_pitch_visual.stl
- link right_knee_pitch: geometry collision cylinder length=0.12 radius=0.045; visual mesh filename=../meshes/visual/right_knee_pitch_visual.stl

File: robots/lite_biped/xacro/lite_biped.description.xacro (robot description, xacro)
@@ -96,7 +96,7 @@
       <!-- Part left_knee_pitch_parts -->
       <collision>
-        <origin xyz="-0.01 0.17 0" rpy="1.5708 1.5708 0" />
-        <geometry>
-          <cylinder length="0.16" radius="0.045" />
+        <origin xyz="-0.015 0.19 0" rpy="1.5708 1.5708 0" />
+        <geometry>
+          <cylinder length="0.12" radius="0.045" />
         </geometry>
       </collision>
@@ -156,5 +156,5 @@
       <!-- Part left_foot_parts -->
       <collision>
-        <origin xyz="0 0.08 0.015" rpy="1.5708 0 0" />
+        <origin xyz="0 0.05 0.015" rpy="1.5708 0 0" />
         <geometry>
           <box size="0.065 0.12 0.03" />
@@ -162,5 +162,5 @@
       </collision>
       <collision>
-        <origin xyz="0 0.07 0.11" rpy="1.91986 0 0" />
+        <origin xyz="0 0.04 0.11" rpy="1.91986 0 0" />
         <geometry>
           <box size="0.07 0.05 0.03" />
@@ -309,7 +309,7 @@
       <!-- Part right_knee_pitch_parts -->
       <collision>
-        <origin xyz="-0.01 0.17 0" rpy="1.5708 1.5708 0" />
-        <geometry>
-          <cylinder length="0.16" radius="0.045" />
+        <origin xyz="-0.015 0.19 0" rpy="1.5708 1.5708 0" />
+        <geometry>
+          <cylinder length="0.12" radius="0.045" />
         </geometry>
       </collision>
@@ -369,5 +369,5 @@
       <!-- Part right_foot_parts -->
       <collision>
-        <origin xyz="0 0.08 0.015" rpy="1.5708 0 -0" />
+        <origin xyz="0 0.05 0.015" rpy="1.5708 0 -0" />
         <geometry>
           <box size="0.065 0.12 0.03" />
@@ -375,5 +375,5 @@
       </collision>
       <collision>
-        <origin xyz="0 0.07 0.11" rpy="1.91986 0 -0" />
+        <origin xyz="0 0.04 0.11" rpy="1.91986 0 -0" />
         <geometry>
           <box size="0.07 0.05 0.03" />

File: robots/lite_pro/urdf/lite_pro.urdf (robot description, URDF)
Before this commit: robot lite_pro, 75 links, 74 joints
Links:
- link left_knee_pitch: geometry collision cylinder length=0.12 radius=0.045; visual mesh filename=../meshes/visual/left_knee_pitch_visual.stl
- link right_knee_pitch: geometry collision cylinder length=0.12 radius=0.045; visual mesh filename=../meshes/visual/right_knee_pitch_visual.stl

File: robots/lite_pro/xacro/lite_pro.description.xacro (robot description, xacro)
@@ -102,7 +102,7 @@
       <!-- Part left_knee_pitch_parts -->
       <collision>
-        <origin xyz="-0.01 0.17 0" rpy="1.5708 1.5708 0" />
-        <geometry>
-          <cylinder length="0.16" radius="0.045" />
+        <origin xyz="-0.015 0.19 0" rpy="1.5708 1.5708 0" />
+        <geometry>
+          <cylinder length="0.12" radius="0.045" />
         </geometry>
       </collision>
@@ -162,5 +162,5 @@
       <!-- Part left_foot_parts -->
       <collision>
-        <origin xyz="0 0.08 0.015" rpy="1.5708 0 0" />
+        <origin xyz="0 0.05 0.015" rpy="1.5708 0 0" />
         <geometry>
           <box size="0.065 0.12 0.03" />
@@ -168,5 +168,5 @@
       </collision>
       <collision>
-        <origin xyz="0 0.07 0.11" rpy="1.91986 0 0" />
+        <origin xyz="0 0.04 0.11" rpy="1.91986 0 0" />
         <geometry>
           <box size="0.07 0.05 0.03" />
@@ -315,7 +315,7 @@
       <!-- Part right_knee_pitch_parts -->
       <collision>
-        <origin xyz="-0.01 0.17 0" rpy="1.5708 1.5708 0" />
-        <geometry>
-          <cylinder length="0.16" radius="0.045" />
+        <origin xyz="-0.015 0.19 0" rpy="1.5708 1.5708 0" />
+        <geometry>
+          <cylinder length="0.12" radius="0.045" />
         </geometry>
       </collision>
@@ -375,5 +375,5 @@
       <!-- Part right_foot_parts -->
       <collision>
-        <origin xyz="0 0.08 0.015" rpy="1.5708 0 -0" />
+        <origin xyz="0 0.05 0.015" rpy="1.5708 0 -0" />
         <geometry>
           <box size="0.065 0.12 0.03" />
@@ -381,5 +381,5 @@
       </collision>
       <collision>
-        <origin xyz="0 0.07 0.11" rpy="1.91986 0 -0" />
+        <origin xyz="0 0.04 0.11" rpy="1.91986 0 -0" />
         <geometry>
           <box size="0.07 0.05 0.03" />
