Commit message: lite_biped: set link masses from measured 3D-printed parts
Regenerated the lite_biped description from the updated Onshape CAD export.
Every biped link's mass is now annotated from the actual 3D-printed part,
replacing the CAD default estimates:

  link           old ->  new (kg)
  pelvis        3.97182 -> 2.10
  hip_pitch     0.61944 -> 0.18
  hip_roll      1.30369 -> 0.93
  hip_yaw       2.08958 -> 1.54
  knee_pitch    0.43540 -> 0.23
  ankle_yaw     1.43174 -> 1.03
  ankle_pitch   0.18412 -> 0.34
  foot          1.20654 -> 0.44
  total (both legs + pelvis)  18.49 -> 11.48

Inertia scales proportionally with each mass override about the unchanged
COM. The pelvis visual mesh is also refreshed (+716 tris) from this export;
all other meshes are geometrically unchanged.

Regenerated offline from the export's robot.pkl (onshape-to-robot --convert)
+ finalize-urdf + mjcf + xacro. All 1376 tests pass.

Co-Authored-By: Claude Opus 4.8 (1M context) <noreply@anthropic.com>

File: robots/lite_biped/urdf/lite_biped.urdf (robot description, URDF)
Before this commit: robot lite_biped, 15 links, 14 joints
Links:
- link left_ankle_pitch: mass 0.184118 -> 0.34
- link left_ankle_yaw: mass 1.43174 -> 1.03
- link left_foot: mass 1.20654 -> 0.44
- link left_hip_pitch: mass 0.619442 -> 0.18
- link left_hip_roll: mass 1.30369 -> 0.93
- link left_hip_yaw: mass 2.08958 -> 1.54
- link left_knee_pitch: mass 0.435399 -> 0.23
- link pelvis: mass 3.97182 -> 2.1
- link right_ankle_pitch: mass 0.184118 -> 0.34
- link right_ankle_yaw: mass 1.43169 -> 1.03
- link right_foot: mass 1.20654 -> 0.44
- link right_hip_pitch: mass 0.619423 -> 0.18
- link right_hip_roll: mass 1.30368 -> 0.93
- link right_hip_yaw: mass 2.08959 -> 1.54
- link right_knee_pitch: mass 0.435358 -> 0.23
Joints:
- joint right_ankle_pitch: origin xyz=0.01 0 -0.34 rpy=-1.5708 -0 -0 -> xyz=0.01 0 -0.34 rpy=-1.5708 0 -0
- joint right_ankle_roll: origin xyz=0 0.04 0 rpy=0 1.5708 0 -> xyz=0 0.04 -0 rpy=0 1.5708 0
- joint right_ankle_yaw: origin xyz=-0.015 0 0 rpy=1.5708 -0 -0 -> xyz=-0.015 0 0 rpy=1.5708 0 -0
- joint right_hip_yaw: origin xyz=0 -0.0068404 -0.0187939 rpy=0 -1.22173 1.5708 -> xyz=-0 -0.0068404 -0.0187939 rpy=0 -1.22173 1.5708
- joint right_knee_pitch: origin xyz=-0.01 -0 -0.33 rpy=-1.5708 0 -0 -> xyz=-0.01 -0 -0.33 rpy=-1.5708 0 0

File: robots/lite_biped/xacro/lite_biped.description.xacro (robot description, xacro)
@@ -12,11 +12,11 @@
     <link name="pelvis">
       <inertial>
-        <origin xyz="0.0135183 5.78646e-07 0.0691358" rpy="0 0 0" />
-        <mass value="3.97182" />
-        <inertia ixx="0.0186861" ixy="7.2433e-08" ixz="-0.000228382" iyy="0.015546" iyz="-9.5463e-08" izz="0.0121371" />
+        <origin xyz="0.0137049 6.97587e-07 0.0692011" rpy="0 0 0" />
+        <mass value="2.1" />
+        <inertia ixx="0.00987937" ixy="3.9803e-08" ixz="-0.000115563" iyy="0.00823366" iyz="-5.1965e-08" izz="0.00638151" />
       </inertial>
       <!-- Part pelvis_parts -->
       <visual>
-        <origin xyz="0.0135183 5.78646e-07 0.0691358" rpy="0 -0 0" />
+        <origin xyz="0.0137049 6.97587e-07 0.0692011" rpy="0 -0 0" />
         <geometry>
           <mesh filename="${mesh_root}/pelvis_visual.stl" />
@@ -31,6 +31,6 @@
       <inertial>
         <origin xyz="-0.0114774 0.00418673 0.0187959" rpy="0 0 0" />
-        <mass value="0.619442" />
-        <inertia ixx="0.000652303" ixy="5.37205e-05" ixz="-0.00011886" iyy="0.000778993" iyz="4.47861e-05" izz="0.000986073" />
+        <mass value="0.18" />
+        <inertia ixx="0.000189549" ixy="1.56103e-05" ixz="-3.45388e-05" iyy="0.000226363" iyz="1.30141e-05" izz="0.000286537" />
       </inertial>
       <!-- Part left_hip_pitch_parts -->
@@ -49,6 +49,6 @@
       <inertial>
         <origin xyz="-4.8952e-08 0.0525082 -0.0652484" rpy="0 0 0" />
-        <mass value="1.30369" />
-        <inertia ixx="0.00368883" ixy="-7.197e-09" ixz="4.838e-09" iyy="0.00199601" iyz="-0.000913168" izz="0.00358153" />
+        <mass value="0.93" />
+        <inertia ixx="0.00263146" ixy="-5.134e-09" ixz="3.451e-09" iyy="0.00142387" iyz="-0.000651416" izz="0.00255491" />
       </inertial>
       <!-- Part left_hip_roll_parts -->
@@ -73,6 +73,6 @@
       <inertial>
         <origin xyz="0.00130442 -2.2783e-05 -0.237299" rpy="0 0 0" />
-        <mass value="2.08958" />
-        <inertia ixx="0.0116205" ixy="1.09303e-06" ixz="-0.000458028" iyy="0.0118686" iyz="2.21073e-07" izz="0.00261694" />
+        <mass value="1.54" />
+        <inertia ixx="0.00856423" ixy="8.05553e-07" ixz="-0.000337563" iyy="0.00874707" iyz="1.62929e-07" izz="0.00192866" />
       </inertial>
       <!-- Part left_hip_yaw_parts -->
@@ -91,6 +91,6 @@
       <inertial>
         <origin xyz="-0.00486713 0.0372163 -0.000224083" rpy="0 0 0" />
-        <mass value="0.435399" />
-        <inertia ixx="0.000913317" ixy="6.65453e-05" ixz="-2.2735e-07" iyy="0.000625586" iyz="1.07178e-06" izz="0.000714736" />
+        <mass value="0.23" />
+        <inertia ixx="0.00048246" ixy="3.51526e-05" ixz="-1.20098e-07" iyy="0.000330466" iyz="5.6617e-07" izz="0.00037756" />
       </inertial>
       <!-- Part left_knee_pitch_parts -->
@@ -115,6 +115,6 @@
       <inertial>
         <origin xyz="-0.00304992 0.00150525 -0.18535" rpy="0 0 0" />
-        <mass value="1.43174" />
-        <inertia ixx="0.00763083" ixy="3.0411e-06" ixz="0.000159775" iyy="0.00768647" iyz="-2.6083e-05" izz="0.00115305" />
+        <mass value="1.03" />
+        <inertia ixx="0.00548966" ixy="2.18778e-06" ixz="0.000114943" iyy="0.00552969" iyz="-1.87643e-05" izz="0.000829513" />
       </inertial>
       <!-- Part left_ankle_yaw_parts -->
@@ -133,6 +133,6 @@
       <inertial>
         <origin xyz="-0.00384209 0.0297371 3.1356e-08" rpy="0 0 0" />
-        <mass value="0.184118" />
-        <inertia ixx="9.75514e-05" ixy="-1.6796e-05" ixz="-4.2e-11" iyy="7.7573e-05" iyz="1.44e-10" izz="0.00013275" />
+        <mass value="0.34" />
+        <inertia ixx="0.000180143" ixy="-3.10163e-05" ixz="-7.8e-11" iyy="0.00014325" iyz="2.66e-10" izz="0.000245142" />
       </inertial>
       <!-- Part left_ankle_pitch_parts -->
@@ -151,6 +151,6 @@
       <inertial>
         <origin xyz="0.00124938 0.0227876 0.0398042" rpy="0 0 0" />
-        <mass value="1.20654" />
-        <inertia ixx="0.00367026" ixy="-9.09996e-06" ixz="-0.000117811" iyy="0.00327589" iyz="-0.000424612" izz="0.00132106" />
+        <mass value="0.44" />
+        <inertia ixx="0.00133847" ixy="-3.31857e-06" ixz="-4.29633e-05" iyy="0.00119465" iyz="-0.000154848" izz="0.000481763" />
       </inertial>
       <!-- Part left_foot_parts -->
@@ -244,6 +244,6 @@
       <inertial>
         <origin xyz="-0.0114771 0.00418737 -0.0187964" rpy="0 0 0" />
-        <mass value="0.619423" />
-        <inertia ixx="0.000652275" ixy="5.37438e-05" ixz="0.000118863" iyy="0.000778995" iyz="-4.4778e-05" izz="0.000986036" />
+        <mass value="0.18" />
+        <inertia ixx="0.000189546" ixy="1.56176e-05" ixz="3.45408e-05" iyy="0.00022637" iyz="-1.30122e-05" izz="0.000286535" />
       </inertial>
       <!-- Part right_hip_pitch_parts -->
@@ -262,6 +262,6 @@
       <inertial>
         <origin xyz="-1.13349e-07 0.0525083 -0.0652488" rpy="0 0 0" />
-        <mass value="1.30368" />
-        <inertia ixx="0.0036888" ixy="3.8e-10" ixz="8.521e-09" iyy="0.00199598" iyz="-0.000913166" izz="0.0035815" />
+        <mass value="0.93" />
+        <inertia ixx="0.00263147" ixy="2.71e-10" ixz="6.079e-09" iyy="0.00142387" iyz="-0.000651423" izz="0.00255493" />
       </inertial>
       <!-- Part right_hip_roll_parts -->
@@ -286,6 +286,6 @@
       <inertial>
         <origin xyz="0.00130421 2.35733e-05 -0.237299" rpy="0 0 0" />
-        <mass value="2.08959" />
-        <inertia ixx="0.0116206" ixy="-1.08279e-06" ixz="-0.000458016" iyy="0.0118687" iyz="-3.03522e-07" izz="0.00261696" />
+        <mass value="1.54" />
+        <inertia ixx="0.00856421" ixy="-7.98006e-07" ixz="-0.000337552" iyy="0.00874705" iyz="-2.23692e-07" izz="0.00192867" />
       </inertial>
       <!-- Part right_hip_yaw_parts -->
@@ -304,6 +304,6 @@
       <inertial>
         <origin xyz="-0.0048642 0.0372186 0.000224747" rpy="0 0 0" />
-        <mass value="0.435358" />
-        <inertia ixx="0.000913266" ixy="6.65739e-05" ixz="2.14089e-07" iyy="0.000625521" iyz="-1.04876e-06" izz="0.00071467" />
+        <mass value="0.23" />
+        <inertia ixx="0.000482479" ixy="3.5171e-05" ixz="1.13103e-07" iyy="0.000330463" iyz="-5.54061e-07" izz="0.000377561" />
       </inertial>
       <!-- Part right_knee_pitch_parts -->
@@ -328,10 +328,10 @@
       <inertial>
         <origin xyz="-0.00304908 -0.0015054 -0.185348" rpy="0 0 0" />
-        <mass value="1.43169" />
-        <inertia ixx="0.00763064" ixy="-3.05072e-06" ixz="0.000159784" iyy="0.00768622" iyz="2.60897e-05" izz="0.00115301" />
+        <mass value="1.03" />
+        <inertia ixx="0.00548969" ixy="-2.19478e-06" ixz="0.000114953" iyy="0.00552968" iyz="1.87697e-05" izz="0.00082951" />
       </inertial>
       <!-- Part right_ankle_yaw_parts -->
       <visual>
-        <origin xyz="-0.00304908 -0.0015054 -0.185348" rpy="-0 0 0" />
+        <origin xyz="-0.00304908 -0.0015054 -0.185348" rpy="0 0 0" />
         <geometry>
           <mesh filename="${mesh_root}/right_ankle_yaw_visual.stl" />
@@ -346,6 +346,6 @@
       <inertial>
         <origin xyz="-0.00384209 0.0297371 3.1396e-08" rpy="0 0 0" />
-        <mass value="0.184118" />
-        <inertia ixx="9.75514e-05" ixy="-1.6796e-05" ixz="-4.2e-11" iyy="7.7573e-05" iyz="1.44e-10" izz="0.00013275" />
+        <mass value="0.34" />
+        <inertia ixx="0.000180143" ixy="-3.10163e-05" ixz="-7.8e-11" iyy="0.00014325" iyz="2.66e-10" izz="0.000245142" />
       </inertial>
       <!-- Part right_ankle_pitch_parts -->
@@ -364,6 +364,6 @@
       <inertial>
         <origin xyz="-0.0012494 0.0227876 0.039804" rpy="0 0 0" />
-        <mass value="1.20654" />
-        <inertia ixx="0.00367026" ixy="9.09895e-06" ixz="0.000117812" iyy="0.00327589" iyz="-0.000424612" izz="0.00132106" />
+        <mass value="0.44" />
+        <inertia ixx="0.00133847" ixy="3.3182e-06" ixz="4.29635e-05" iyy="0.00119465" iyz="-0.000154847" izz="0.000481763" />
       </inertial>
       <!-- Part right_foot_parts -->
@@ -392,5 +392,5 @@
     <!-- Joint from right_ankle_pitch to right_foot -->
     <joint name="right_ankle_roll" type="revolute">
-      <origin xyz="0 0.04 0" rpy="0 1.5708 0" />
+      <origin xyz="0 0.04 -0" rpy="0 1.5708 0" />
       <parent link="right_ankle_pitch" />
       <child link="right_foot" />
@@ -401,5 +401,5 @@
     <!-- Joint from right_ankle_yaw to right_ankle_pitch -->
     <joint name="right_ankle_pitch" type="revolute">
-      <origin xyz="0.01 0 -0.34" rpy="-1.5708 -0 -0" />
+      <origin xyz="0.01 0 -0.34" rpy="-1.5708 0 -0" />
       <parent link="right_ankle_yaw" />
       <child link="right_ankle_pitch" />
@@ -410,5 +410,5 @@
     <!-- Joint from right_knee_pitch to right_ankle_yaw -->
     <joint name="right_ankle_yaw" type="revolute">
-      <origin xyz="-0.015 0 0" rpy="1.5708 -0 -0" />
+      <origin xyz="-0.015 0 0" rpy="1.5708 0 -0" />
       <parent link="right_knee_pitch" />
       <child link="right_ankle_yaw" />
@@ -419,5 +419,5 @@
     <!-- Joint from right_hip_yaw to right_knee_pitch -->
     <joint name="right_knee_pitch" type="revolute">
-      <origin xyz="-0.01 -0 -0.33" rpy="-1.5708 0 -0" />
+      <origin xyz="-0.01 -0 -0.33" rpy="-1.5708 0 0" />
       <parent link="right_hip_yaw" />
       <child link="right_knee_pitch" />
@@ -428,5 +428,5 @@
     <!-- Joint from right_hip_roll to right_hip_yaw -->
     <joint name="right_hip_yaw" type="revolute">
-      <origin xyz="0 -0.0068404 -0.0187939" rpy="0 -1.22173 1.5708" />
+      <origin xyz="-0 -0.0068404 -0.0187939" rpy="0 -1.22173 1.5708" />
       <parent link="right_hip_roll" />
       <child link="right_hip_yaw" />

Commit message: lite_biped: add IMU frame (pelvis +0.08 m) from CAD re-export
Re-exported the Biped assembly from Onshape. Adds an `imu` frame — a
massless link fixed to `pelvis` at z=+0.08 m with identity orientation —
marking the true IMU mounting point (previously unspecified, so consumers
placed the IMU at the pelvis origin). Colliders (4 box + 4 capsule),
link masses, and joints are otherwise unchanged from the previous release.

Co-Authored-By: Claude Opus 4.8 (1M context) <noreply@anthropic.com>
Claude-Session: https://claude.ai/code/session_01Ld2SFYRAtw46paSDdG5qT4

File: robots/lite_biped/urdf/lite_biped.urdf (robot description, URDF)
Before this commit: robot lite_biped, 15 links, 14 joints
Links:
- added link imu, mass 1e-9
Joints:
- added joint imu_frame: type fixed, parent pelvis, child imu, origin xyz=0 0 0.08 rpy=0 -0 0, axis 0 0 0
- joint right_ankle_pitch: origin xyz=0.01 0 -0.34 rpy=-1.5708 0 -0 -> xyz=0.01 0 -0.34 rpy=-1.5708 0 0
- joint right_ankle_roll: origin xyz=0 0.04 -0 rpy=0 1.5708 0 -> xyz=-0 0.04 -0 rpy=-0 1.5708 0
- joint right_ankle_yaw: origin xyz=-0.015 0 0 rpy=1.5708 0 -0 -> xyz=-0.015 0 -0 rpy=1.5708 -0 -0

File: robots/lite_biped/xacro/lite_biped.description.xacro (robot description, xacro)
@@ -27,4 +27,19 @@
       </visual>
     </link>
+    <!-- Frame imu (dummy link + fixed joint) -->
+    <link name="imu">
+      <origin xyz="0 0 0" rpy="0 -0 0" />
+      <inertial>
+        <origin xyz="0 0 0" rpy="0 0 0" />
+        <mass value="1e-9" />
+        <inertia ixx="0" ixy="0" ixz="0" iyy="0" iyz="0" izz="0" />
+      </inertial>
+    </link>
+    <joint name="imu_frame" type="fixed">
+      <origin xyz="0 0 0.08" rpy="0 -0 0" />
+      <parent link="pelvis" />
+      <child link="imu" />
+      <axis xyz="0 0 0" />
+    </joint>
     <!-- Link left_hip_pitch -->
     <link name="left_hip_pitch">
@@ -392,5 +407,5 @@
     <!-- Joint from right_ankle_pitch to right_foot -->
     <joint name="right_ankle_roll" type="revolute">
-      <origin xyz="0 0.04 -0" rpy="0 1.5708 0" />
+      <origin xyz="-0 0.04 -0" rpy="-0 1.5708 0" />
       <parent link="right_ankle_pitch" />
       <child link="right_foot" />
@@ -401,5 +416,5 @@
     <!-- Joint from right_ankle_yaw to right_ankle_pitch -->
     <joint name="right_ankle_pitch" type="revolute">
-      <origin xyz="0.01 0 -0.34" rpy="-1.5708 0 -0" />
+      <origin xyz="0.01 0 -0.34" rpy="-1.5708 0 0" />
       <parent link="right_ankle_yaw" />
       <child link="right_ankle_pitch" />
@@ -410,5 +425,5 @@
     <!-- Joint from right_knee_pitch to right_ankle_yaw -->
     <joint name="right_ankle_yaw" type="revolute">
-      <origin xyz="-0.015 0 0" rpy="1.5708 0 -0" />
+      <origin xyz="-0.015 0 -0" rpy="1.5708 -0 -0" />
       <parent link="right_knee_pitch" />
       <child link="right_ankle_yaw" />
