Commit message: lite_biped: real leg CAN map + directions, ankle_yaw +/-90deg, IMU at mount
- ros2_control.json: real leg CAN ids from a live bus scan (left can2 31-37,
  right can3 41-47), buses can2/can3, and commissioned joint directions (5
  flipped to -1: left_hip_pitch/knee_pitch/ankle_roll, right_ankle_pitch/
  ankle_roll -- verified in the viewer against the physical robot).
- ankle_yaw limit +/-45deg -> +/-90deg from the updated CAD export (matches the
  real hardware range). Regenerated urdf/mjcf/xacro from the export's robot.pkl.
- IMU: the new CAD adds an `imu` link at the real mount (pelvis+0.08); kept it and
  moved the sim imu_site + base sensors there (physics.json imu.pos) so the sim
  IMU sits where the real one is.

Co-Authored-By: Claude Opus 4.8 (1M context) <noreply@anthropic.com>
Claude-Session: https://claude.ai/code/session_019QrgD2S2yba6bDj4wzGWeB

File: robots/lite_biped/urdf/lite_biped.urdf (robot description, URDF)
Before this commit: robot lite_biped, 15 links, 14 joints
Links:
- added link imu, mass 1e-9
Joints:
- added joint imu_frame: type fixed, parent pelvis, child imu, origin xyz=0 0 0.08 rpy=0 -0 0, axis 0 0 0
- joint left_ankle_yaw: limit lower=-0.785398 upper=0.785398 effort=14.0 velocity=100 -> lower=-1.5708 upper=1.5708 effort=14.0 velocity=100
- joint right_ankle_pitch: origin xyz=0.01 0 -0.34 rpy=-1.5708 0 -0 -> xyz=0.01 0 -0.34 rpy=-1.5708 0 0
- joint right_ankle_roll: origin xyz=0 0.04 -0 rpy=0 1.5708 0 -> xyz=0 0.04 -0 rpy=-0 1.5708 0
- joint right_ankle_yaw: limit lower=-0.785398 upper=0.785398 effort=14.0 velocity=100 -> lower=-1.5708 upper=1.5708 effort=14.0 velocity=100; origin xyz=-0.015 0 0 rpy=1.5708 0 -0 -> xyz=-0.015 0 0 rpy=1.5708 -0 -0
- joint right_hip_yaw: origin xyz=-0 -0.0068404 -0.0187939 rpy=0 -1.22173 1.5708 -> xyz=0 -0.0068404 -0.0187939 rpy=0 -1.22173 1.5708
- joint right_knee_pitch: origin xyz=-0.01 -0 -0.33 rpy=-1.5708 0 0 -> xyz=-0.01 -0 -0.33 rpy=-1.5708 -0 0

File: robots/lite_biped/xacro/lite_biped.description.xacro (robot description, xacro)
@@ -27,4 +27,19 @@
       </visual>
     </link>
+    <!-- Frame imu (dummy link + fixed joint) -->
+    <link name="imu">
+      <origin xyz="0 0 0" rpy="0 -0 0" />
+      <inertial>
+        <origin xyz="0 0 0" rpy="0 0 0" />
+        <mass value="1e-9" />
+        <inertia ixx="0" ixy="0" ixz="0" iyy="0" iyz="0" izz="0" />
+      </inertial>
+    </link>
+    <joint name="imu_frame" type="fixed">
+      <origin xyz="0 0 0.08" rpy="0 -0 0" />
+      <parent link="pelvis" />
+      <child link="imu" />
+      <axis xyz="0 0 0" />
+    </joint>
     <!-- Link left_hip_pitch -->
     <link name="left_hip_pitch">
@@ -201,5 +216,5 @@
       <child link="left_ankle_yaw" />
       <axis xyz="0 0 1" />
-      <limit effort="14.0" velocity="100" lower="-0.785398" upper="0.785398" />
+      <limit effort="14.0" velocity="100" lower="-1.5708" upper="1.5708" />
       <joint_properties friction="0.1" />
     </joint>
@@ -261,5 +276,5 @@
     <link name="right_hip_roll">
       <inertial>
-        <origin xyz="-1.13349e-07 0.0525083 -0.0652488" rpy="0 0 0" />
+        <origin xyz="2.6715e-08 0.0525085 -0.0652483" rpy="0 0 0" />
         <mass value="0.93" />
         <inertia ixx="0.00263147" ixy="2.71e-10" ixz="6.079e-09" iyy="0.00142387" iyz="-0.000651423" izz="0.00255493" />
@@ -267,5 +282,5 @@
       <!-- Part right_hip_roll_parts -->
       <collision>
-        <origin xyz="-0 0.181098 -0.0871979" rpy="1.22173 0 0" />
+        <origin xyz="1.40064e-07 0.181098 -0.0871974" rpy="1.22173 -0 0" />
         <geometry>
           <cylinder length="0.15" radius="0.05" />
@@ -273,5 +288,5 @@
       </collision>
       <visual>
-        <origin xyz="-1.13349e-07 0.0525083 -0.0652488" rpy="0 -1.22173 1.5708" />
+        <origin xyz="2.6715e-08 0.0525085 -0.0652483" rpy="0 -1.22173 1.5708" />
         <geometry>
           <mesh filename="${mesh_root}/right_hip_roll_visual.stl" />
@@ -291,5 +306,5 @@
       <!-- Part right_hip_yaw_parts -->
       <visual>
-        <origin xyz="0.00130421 2.35733e-05 -0.237299" rpy="0 0 0" />
+        <origin xyz="0.00130421 2.35733e-05 -0.237299" rpy="0 -0 0" />
         <geometry>
           <mesh filename="${mesh_root}/right_hip_yaw_visual.stl" />
@@ -392,5 +407,5 @@
     <!-- Joint from right_ankle_pitch to right_foot -->
     <joint name="right_ankle_roll" type="revolute">
-      <origin xyz="0 0.04 -0" rpy="0 1.5708 0" />
+      <origin xyz="0 0.04 -0" rpy="-0 1.5708 0" />
       <parent link="right_ankle_pitch" />
       <child link="right_foot" />
@@ -401,5 +416,5 @@
     <!-- Joint from right_ankle_yaw to right_ankle_pitch -->
     <joint name="right_ankle_pitch" type="revolute">
-      <origin xyz="0.01 0 -0.34" rpy="-1.5708 0 -0" />
+      <origin xyz="0.01 0 -0.34" rpy="-1.5708 0 0" />
       <parent link="right_ankle_yaw" />
       <child link="right_ankle_pitch" />
@@ -410,14 +425,14 @@
     <!-- Joint from right_knee_pitch to right_ankle_yaw -->
     <joint name="right_ankle_yaw" type="revolute">
-      <origin xyz="-0.015 0 0" rpy="1.5708 0 -0" />
+      <origin xyz="-0.015 0 0" rpy="1.5708 -0 -0" />
       <parent link="right_knee_pitch" />
       <child link="right_ankle_yaw" />
       <axis xyz="0 0 1" />
-      <limit effort="14.0" velocity="100" lower="-0.785398" upper="0.785398" />
+      <limit effort="14.0" velocity="100" lower="-1.5708" upper="1.5708" />
       <joint_properties friction="0.1" />
     </joint>
     <!-- Joint from right_hip_yaw to right_knee_pitch -->
     <joint name="right_knee_pitch" type="revolute">
-      <origin xyz="-0.01 -0 -0.33" rpy="-1.5708 0 0" />
+      <origin xyz="-0.01 -0 -0.33" rpy="-1.5708 -0 0" />
       <parent link="right_hip_yaw" />
       <child link="right_knee_pitch" />
@@ -428,5 +443,5 @@
     <!-- Joint from right_hip_roll to right_hip_yaw -->
     <joint name="right_hip_yaw" type="revolute">
-      <origin xyz="-0 -0.0068404 -0.0187939" rpy="0 -1.22173 1.5708" />
+      <origin xyz="0 -0.0068404 -0.0187939" rpy="0 -1.22173 1.5708" />
       <parent link="right_hip_roll" />
       <child link="right_hip_yaw" />

File: robots/lite_biped/xacro/lite_biped.ros2_control.xacro (robot description, xacro)
@@ -29,29 +29,29 @@
   </xacro:macro>
   <xacro:macro name="lite_biped_left_leg_joints" params="use_fake_hardware use_sim">
-    <xacro:lite_biped_joint name="left_hip_pitch" can_id="11" model="rs-06" direction="1"
+    <xacro:lite_biped_joint name="left_hip_pitch" can_id="31" model="rs-06" direction="-1"
                       lower_limit="-2.35619" upper_limit="0.785398"
                       torque_limit="36.0" current_limit="43"
                       use_fake_hardware="${use_fake_hardware}" use_sim="${use_sim}"/>
-    <xacro:lite_biped_joint name="left_hip_roll" can_id="12" model="rs-06" direction="1"
+    <xacro:lite_biped_joint name="left_hip_roll" can_id="32" model="rs-06" direction="1"
                       lower_limit="-0.349066" upper_limit="1.5708"
                       torque_limit="36.0" current_limit="43"
                       use_fake_hardware="${use_fake_hardware}" use_sim="${use_sim}"/>
-    <xacro:lite_biped_joint name="left_hip_yaw" can_id="13" model="rs-02" direction="1"
+    <xacro:lite_biped_joint name="left_hip_yaw" can_id="33" model="rs-02" direction="1"
                       lower_limit="-1.5708" upper_limit="1.5708"
                       torque_limit="17.0" current_limit="27"
                       use_fake_hardware="${use_fake_hardware}" use_sim="${use_sim}"/>
-    <xacro:lite_biped_joint name="left_knee_pitch" can_id="14" model="rs-06" direction="1"
+    <xacro:lite_biped_joint name="left_knee_pitch" can_id="34" model="rs-06" direction="-1"
                       lower_limit="0.0" upper_limit="2.35619"
                       torque_limit="36.0" current_limit="43"
                       use_fake_hardware="${use_fake_hardware}" use_sim="${use_sim}"/>
-    <xacro:lite_biped_joint name="left_ankle_yaw" can_id="15" model="rs-00" direction="1"
-                      lower_limit="-0.785398" upper_limit="0.785398"
+    <xacro:lite_biped_joint name="left_ankle_yaw" can_id="35" model="rs-00" direction="1"
+                      lower_limit="-1.5708" upper_limit="1.5708"
                       torque_limit="14.0" current_limit="16"
                       use_fake_hardware="${use_fake_hardware}" use_sim="${use_sim}"/>
-    <xacro:lite_biped_joint name="left_ankle_pitch" can_id="16" model="rs-00" direction="1"
+    <xacro:lite_biped_joint name="left_ankle_pitch" can_id="36" model="rs-00" direction="1"
                       lower_limit="-0.523599" upper_limit="0.872665"
                       torque_limit="14.0" current_limit="16"
                       use_fake_hardware="${use_fake_hardware}" use_sim="${use_sim}"/>
-    <xacro:lite_biped_joint name="left_ankle_roll" can_id="17" model="rs-05" direction="1"
+    <xacro:lite_biped_joint name="left_ankle_roll" can_id="37" model="rs-05" direction="-1"
                       lower_limit="-0.349066" upper_limit="0.349066"
                       torque_limit="5.5" current_limit="14"
@@ -59,29 +59,29 @@
   </xacro:macro>
   <xacro:macro name="lite_biped_right_leg_joints" params="use_fake_hardware use_sim">
-    <xacro:lite_biped_joint name="right_hip_pitch" can_id="21" model="rs-06" direction="1"
+    <xacro:lite_biped_joint name="right_hip_pitch" can_id="41" model="rs-06" direction="1"
                       lower_limit="-2.35619" upper_limit="0.785398"
                       torque_limit="36.0" current_limit="43"
                       use_fake_hardware="${use_fake_hardware}" use_sim="${use_sim}"/>
-    <xacro:lite_biped_joint name="right_hip_roll" can_id="22" model="rs-06" direction="1"
+    <xacro:lite_biped_joint name="right_hip_roll" can_id="42" model="rs-06" direction="1"
                       lower_limit="-1.5708" upper_limit="0.349066"
                       torque_limit="36.0" current_limit="43"
                       use_fake_hardware="${use_fake_hardware}" use_sim="${use_sim}"/>
-    <xacro:lite_biped_joint name="right_hip_yaw" can_id="23" model="rs-02" direction="1"
+    <xacro:lite_biped_joint name="right_hip_yaw" can_id="43" model="rs-02" direction="1"
                       lower_limit="-1.5708" upper_limit="1.5708"
                       torque_limit="17.0" current_limit="27"
                       use_fake_hardware="${use_fake_hardware}" use_sim="${use_sim}"/>
-    <xacro:lite_biped_joint name="right_knee_pitch" can_id="24" model="rs-06" direction="1"
+    <xacro:lite_biped_joint name="right_knee_pitch" can_id="44" model="rs-06" direction="1"
                       lower_limit="0.0" upper_limit="2.35619"
                       torque_limit="36.0" current_limit="43"
                       use_fake_hardware="${use_fake_hardware}" use_sim="${use_sim}"/>
-    <xacro:lite_biped_joint name="right_ankle_yaw" can_id="25" model="rs-00" direction="1"
-                      lower_limit="-0.785398" upper_limit="0.785398"
+    <xacro:lite_biped_joint name="right_ankle_yaw" can_id="45" model="rs-00" direction="1"
+                      lower_limit="-1.5708" upper_limit="1.5708"
                       torque_limit="14.0" current_limit="16"
                       use_fake_hardware="${use_fake_hardware}" use_sim="${use_sim}"/>
-    <xacro:lite_biped_joint name="right_ankle_pitch" can_id="26" model="rs-00" direction="1"
+    <xacro:lite_biped_joint name="right_ankle_pitch" can_id="46" model="rs-00" direction="-1"
                       lower_limit="-0.523599" upper_limit="0.872665"
                       torque_limit="14.0" current_limit="16"
                       use_fake_hardware="${use_fake_hardware}" use_sim="${use_sim}"/>
-    <xacro:lite_biped_joint name="right_ankle_roll" can_id="27" model="rs-05" direction="1"
+    <xacro:lite_biped_joint name="right_ankle_roll" can_id="47" model="rs-05" direction="-1"
                       lower_limit="-0.349066" upper_limit="0.349066"
                       torque_limit="5.5" current_limit="14"

File: robots/lite_biped/xacro/lite_biped.urdf.xacro (robot description, xacro)
@@ -5,6 +5,6 @@
   <xacro:arg name="use_sim" default="false"/>
   <xacro:arg name="mode" default="legs"/>
-  <xacro:arg name="can_interface_left" default="can0"/>
-  <xacro:arg name="can_interface_right" default="can1"/>
+  <xacro:arg name="can_interface_left" default="can2"/>
+  <xacro:arg name="can_interface_right" default="can3"/>
   <xacro:arg name="calibration_file" default=""/>
   <xacro:include filename="$(find lite_description)/robots/lite_biped/xacro/lite_biped.description.xacro"/>

Commit message: Feat/lite biped deploy (#10)
* lite_biped: sim deploy asset (freejoint + IMU + contacts) on measured masses

Extend the robot_assets generator and the lite_biped variant to produce a
MuJoCo deploy/sim asset for the biped locomotion stack:

- urdf_to_mjcf: add a floating base, IMU site + accel/gyro/quat/vel/pos sensors,
  and foot-contact patching (foot bodies condim=3 + friction/priority, others
  condim=1), all opt-in per variant via cad/physics.json.
- urdf_to_xacro: emit a base_imu ros2_control sensor block (sim only).
- lite_biped/cad: physics.json (option matched to mjlab: timestep 0.005,
  pyramidal cone, impratio 1, iterations 10/20; + freejoint/imu/contact) and a
  new ros2_control.json (legs + imu).
- lite_biped/mjcf: regenerated lite_biped.xml + hand-authored lite_biped_scene.xml
  (floor + light + `home` standing keyframe at base z=0.80).
- Link masses/inertias now the measured 3D-printed-part values (pelvis 2.1,
  total ~11.48 kg), incorporating Lite-Description 479ed5e -- matches the
  training asset (was outdated CAD masses ~18.5 kg).

Regenerated urdf/xacro/mjcf; 1415 generator tests pass.

Co-Authored-By: Claude Opus 4.8 (1M context) <noreply@anthropic.com>
Claude-Session: https://claude.ai/code/session_019QrgD2S2yba6bDj4wzGWeB

* lite_biped: real leg CAN map + directions, ankle_yaw +/-90deg, IMU at mount

- ros2_control.json: real leg CAN ids from a live bus scan (left can2 31-37,
  right can3 41-47), buses can2/can3, and commissioned joint directions (5
  flipped to -1: left_hip_pitch/knee_pitch/ankle_roll, right_ankle_pitch/
  ankle_roll -- verified in the viewer against the physical robot).
- ankle_yaw limit +/-45deg -> +/-90deg from the updated CAD export (matches the
  real hardware range). Regenerated urdf/mjcf/xacro from the export's robot.pkl.
- IMU: the new CAD adds an `imu` link at the real mount (pelvis+0.08); kept it and
  moved the sim imu_site + base sensors there (physics.json imu.pos) so the sim
  IMU sits where the real one is.

Co-Authored-By: Claude Opus 4.8 (1M context) <noreply@anthropic.com>
Claude-Session: https://claude.ai/code/session_019QrgD2S2yba6bDj4wzGWeB

---------

Co-authored-by: Claude Opus 4.8 (1M context) <noreply@anthropic.com>

File: robots/lite_biped/urdf/lite_biped.urdf (robot description, URDF)
Before this commit: robot lite_biped, 16 links, 15 joints
Joints:
- joint left_ankle_yaw: limit lower=-0.785398 upper=0.785398 effort=14.0 velocity=100 -> lower=-1.5708 upper=1.5708 effort=14.0 velocity=100
- joint right_ankle_yaw: limit lower=-0.785398 upper=0.785398 effort=14.0 velocity=100 -> lower=-1.5708 upper=1.5708 effort=14.0 velocity=100

File: robots/lite_biped/xacro/lite_biped.description.xacro (robot description, xacro)
@@ -216,5 +216,5 @@
       <child link="left_ankle_yaw" />
       <axis xyz="0 0 1" />
-      <limit effort="14.0" velocity="100" lower="-0.785398" upper="0.785398" />
+      <limit effort="14.0" velocity="100" lower="-1.5708" upper="1.5708" />
       <joint_properties friction="0.1" />
     </joint>
@@ -429,5 +429,5 @@
       <child link="right_ankle_yaw" />
       <axis xyz="0 0 1" />
-      <limit effort="14.0" velocity="100" lower="-0.785398" upper="0.785398" />
+      <limit effort="14.0" velocity="100" lower="-1.5708" upper="1.5708" />
       <joint_properties friction="0.1" />
     </joint>

File: robots/lite_biped/xacro/lite_biped.urdf.xacro (robot description, xacro)
@@ -2,5 +2,20 @@
 <!-- GENERATED by robot_assets from Onshape CAD. Do not edit by hand. Regenerate: robot-assets-generate lite_biped -->
 <robot xmlns:xacro="http://www.ros.org/wiki/xacro" name="lite_biped">
+  <xacro:arg name="use_fake_hardware" default="true"/>
+  <xacro:arg name="use_sim" default="false"/>
+  <xacro:arg name="mode" default="legs"/>
+  <xacro:arg name="can_interface_left" default="can2"/>
+  <xacro:arg name="can_interface_right" default="can3"/>
+  <xacro:arg name="calibration_file" default=""/>
   <xacro:include filename="$(find lite_description)/robots/lite_biped/xacro/lite_biped.description.xacro"/>
+  <xacro:include filename="$(find lite_description)/robots/lite_biped/xacro/lite_biped.ros2_control.xacro"/>
   <xacro:lite_biped_description/>
+  <xacro:lite_biped_ros2_control
+    name="LiteBipedHardware"
+    use_fake_hardware="$(arg use_fake_hardware)"
+    use_sim="$(arg use_sim)"
+    mode="$(arg mode)"
+    can_interface_left="$(arg can_interface_left)"
+    can_interface_right="$(arg can_interface_right)"
+    calibration_file="$(arg calibration_file)"/>
 </robot>
